Commit message: Distance/Collision marker visualization in Rviz added

File: morpheus_teleop/config/test_robot.urdf (robot description, URDF)
Before this commit: robot a_bot_scene, 39 links, 38 joints
Links:
- added link test_link, mass 2; collision mesh filename=package://morpheus_teleop/meshes/components/collision/teapo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 scale=.05 .05 .05; visual mesh filename=package://morpheus_teleop/meshes/components/visual/teapot.o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 scale=.05 .05 .05
Joints:
- added joint world_joint: type fixed, parent world, child test_link, origin xyz=0.0 0.0 0.5 rpy=0.0 0.0 0.0
