Commit message: Adding obstacles, removing old test files

File: morpheus_teleop/urdf/macros/table_2x8ft.xacro (robot description, xacro)
@@ -1,7 +1,7 @@
 <?xml version="1.0"?>
-<robot name="double_sided_shelf" xmlns:xacro="http://www.ros.org/wiki/xacro">
-  <xacro:macro name="double_sided_shelf"
+<robot name="table_2x8ft" xmlns:xacro="http://www.ros.org/wiki/xacro">
+  <xacro:macro name="table_2x8ft"
     params="x:=0 y:=0 z:=0 scale:=0.05 prefix parent">
-    <link name="${prefix}double_sided_shelf">
+    <link name="${prefix}table_2x8ft">
         <contact>
             <lateral_friction value="1.0"/>
@@ -18,5 +18,5 @@
             <origin rpy="1.57079632679 0 0" xyz="0 0 0"/>
             <geometry>
-                <mesh filename="package://morpheus_teleop/meshes/components/visual/double_sided_shelf.obj" scale="${scale} ${scale} ${scale}"/>
+                <mesh filename="package://morpheus_teleop/meshes/components/visual/table_2x8ft.obj" scale="${scale} ${scale} ${scale}"/>
             </geometry>
             <material name="grey">
@@ -27,11 +27,11 @@
             <origin rpy="1.57079632679 0 0" xyz="0 0 0" />
             <geometry>
-                <mesh filename="package://morpheus_teleop/meshes/components/collision/double_sided_shelf.obj" scale="${scale} ${scale} ${scale}"/>
+                <mesh filename="package://morpheus_teleop/meshes/components/collision/table_2x8ft.obj" scale="${scale} ${scale} ${scale}"/>
             </geometry>
         </collision>
     </link>
-    <joint name="${prefix}double_sided_shelf_joint" type="fixed">
+    <joint name="${prefix}table_2x8ft_joint" type="fixed">
       <parent link="${parent}" />
-      <child link="${prefix}double_sided_shelf" />
+      <child link="${prefix}table_2x8ft" />
       <origin xyz="${x} ${y} ${z}" />
     </joint>

File: morpheus_teleop/urdf/scenes/a_bot_double_sided_shelf_scene.xacro (robot description, xacro)
@@ -6,9 +6,18 @@
         prefix=""
         parent="world"
-        x="0.5"
-        y="0.0"
+        x="0.0"
+        y="0.6952"
         z="0.5"
         scale="0.0254"
     />
     <!-- scale=0.0254 meters/inch -->
+    <xacro:include filename="$(find morpheus_teleop)/urdf/macros/table_2x8ft.xacro" />
+    <xacro:table_2x8ft
+        prefix=""
+        parent="world"
+        x="-0.5"
+        y="1.0"
+        z="0.5"
+        scale="0.0254"
+    />
 </robot>
