Commit message: Object spawner fixes, obstacle refactoring

File: morpheus_teleop/urdf/macros/bar_12in.xacro (robot description, xacro)
@@ -2,16 +2,16 @@
 <robot name="bar_12in" xmlns:xacro="http://www.ros.org/wiki/xacro">
   <xacro:macro name="bar_12in"
-    params="x:=0 y:=0 z:=0 scale:=0.0254 prefix parent">
+    params="x:=0 y:=0 z:=0 R:=0 P:=0 Y:=0 scale:=0.0254 prefix parent">
     <link name="${prefix}bar_12in">
         <contact>
             <lateral_friction value="1.0"/>
-            <rolling_friction value="0.0"/>
+            <rolling_friction value="0.05"/>
             <contact_cfm value="0.0"/>
             <contact_erp value="1.0"/>
         </contact>
         <inertial>
-            <origin rpy="0 0 0" xyz="${scale * 0.5} ${scale * 0.5} ${scale * 6}"/>
-            <mass value="1"/>
-            <inertia ixx="1" ixy="0" ixz="0" iyy="12" iyz="0" izz="12"/>
+            <origin rpy="0 0 0" xyz="${scale * 0.5} ${scale * 6.0} ${scale * 0.5}"/>
+            <mass value="0.15"/>
+            <inertia ixx="${scale * 12.0}" ixy="0" ixz="0" iyy="${scale * 1.0}" iyz="0" izz="${scale * 12.0}"/>
         </inertial>
         <visual>
@@ -31,4 +31,9 @@
         </collision>
     </link>
+    <joint name="${prefix}bar_12in_joint" type="fixed">
+        <parent link="${parent}" />
+        <child link="${prefix}bar_12in" />
+        <origin xyz="${x} ${y} ${z}" rpy="${R} ${P} ${Y}" />
+    </joint>
   </xacro:macro>
 </robot>

File: morpheus_teleop/urdf/macros/bar_4in.xacro (robot description, xacro)
@@ -2,5 +2,5 @@
 <robot name="bar_4in" xmlns:xacro="http://www.ros.org/wiki/xacro">
   <xacro:macro name="bar_4in"
-    params="x:=0 y:=0 z:=0 scale:=0.0254 prefix parent">
+    params="x:=0 y:=0 z:=0 R:=0 P:=0 Y:=0 scale:=0.0254 prefix parent">
     <link name="${prefix}bar_4in">
         <contact>
@@ -12,5 +12,5 @@
         <inertial>
             <origin rpy="0 0 0" xyz="${scale * 0.5} ${scale * 0.5} ${scale * 2}"/>
-            <mass value="1"/>
+            <mass value="0.05"/>
             <inertia ixx="1" ixy="0" ixz="0" iyy="12" iyz="0" izz="12"/>
         </inertial>
@@ -31,4 +31,9 @@
         </collision>
     </link>
+    <joint name="${prefix}bar_4in_joint" type="fixed">
+        <parent link="${parent}" />
+        <child link="${prefix}bar_4in" />
+        <origin xyz="${x} ${y} ${z}" rpy="${R} ${P} ${Y}" />
+    </joint>
   </xacro:macro>
 </robot>

File: morpheus_teleop/urdf/macros/block.xacro (robot description, xacro)
@@ -2,5 +2,5 @@
 <robot name="block" xmlns:xacro="http://www.ros.org/wiki/xacro">
   <xacro:macro name="block"
-    params="x:=0 y:=0 z:=0 scale:=0.0254 prefix parent">
+    params="x:=0 y:=0 z:=0 R:=0 P:=0 Y:=0 scale:=0.0254 prefix parent">
     <link name="${prefix}block">
         <contact>
@@ -31,4 +31,9 @@
         </collision>
     </link>
+    <joint name="${prefix}block_joint" type="fixed">
+        <parent link="${parent}" />
+        <child link="${prefix}block" />
+        <origin xyz="${x} ${y} ${z}" rpy="${R} ${P} ${Y}" />
+    </joint>
   </xacro:macro>
 </robot>

File: morpheus_teleop/urdf/macros/double_level_shelf.xacro (robot description, xacro)
@@ -3,24 +3,32 @@
   <xacro:include filename="$(find morpheus_teleop)/urdf/macros/shelf.xacro" />
   <xacro:macro name="double_level_shelf"
-    params="x:=0 y:=0 z:=0 scale:=0.0254 prefix parent">
+    params="x:=0 y:=0 z:=0 R:=0 P:=0 Y:=0 scale:=0.0254 prefix parent">
+    <link name="${prefix}double_level_shelf"/>
     <xacro:shelf
+        x="0"
+        y="0"
+        z="0"
+        R="0"
+        P="0"
+        Y="0"
         prefix="${prefix}bottom_"
-        parent="${parent}"
+        parent="${prefix}double_level_shelf"
         scale="${scale}"
     />
     <xacro:shelf
+        x="0"
+        y="0"
+        z="0"
+        R="0"
+        P="0"
+        Y="0"
         prefix="${prefix}top_"
-        parent="${parent}"
+        parent="${prefix}double_level_shelf"
         scale="${scale}"
     />
-    <joint name="${prefix}double_level_shelf_bottom_shelf_joint" type="fixed">
+    <joint name="${prefix}double_level_shelf_joint" type="fixed">
       <parent link="${parent}" />
-      <child link="${prefix}bottom_shelf" />
-      <origin rpy="0 0 0" xyz="${x} ${y} ${z}" />
-    </joint>
-    <joint name="${prefix}double_level_shelf_topshelf_joint" type="fixed">
-      <parent link="${parent}" />
-      <child link="${prefix}top_shelf" />
-      <origin rpy="0 0 0" xyz="${x} ${y} ${scale * 5 + z}" />
+      <child link="${prefix}double_level_shelf" />
+      <origin xyz="${x} ${y} ${z}" rpy="${R} ${P} ${Y}" />
     </joint>
   </xacro:macro>

File: morpheus_teleop/urdf/macros/double_sided_shelf.xacro (robot description, xacro)
@@ -4,44 +4,54 @@
   <xacro:include filename="$(find morpheus_teleop)/urdf/macros/wall_4x12in.xacro" />
   <xacro:macro name="double_sided_shelf"
-    params="x:=0 y:=0 z:=0 scale:=0.0254 prefix parent">
+    params="x:=0 y:=0 z:=0 R:=0 P:=0 Y:=0 scale:=0.0254 prefix parent">
+    <link name="${prefix}double_sided_shelf"/>
     <xacro:shelf
+        x="${scale * 4}"
+        y="0"
+        z="0"
+        R="0"
+        P="0"
+        Y="${pi/2}"
         prefix="${prefix}left_"
-        parent="${parent}"
+        parent="${prefix}double_sided_shelf"
         scale="${scale}"
     />
     <xacro:shelf
+        x="${scale * 9}"
+        y="0"
+        z="0"
+        R="0"
+        P="0"
+        Y="${pi/2}"
         prefix="${prefix}right_"
-        parent="${parent}"
+        parent="${prefix}double_sided_shelf"
         scale="${scale}"
     />
     <xacro:wall_4x12in
+        x="${scale * 4}"
+        y="0"
+        z="0"
+        R="${pi/2}"
+        P="0"
+        Y="${pi/2}"
         prefix="${prefix}bottom_"
-        parent="${parent}"
+        parent="${prefix}double_sided_shelf"
         scale="${scale}"
     />
     <xacro:wall_4x12in
+        x="${scale * 4}"
+        y="0"
+        z="${scale * 4}"
+        R="${pi/2}"
+        P="0"
+        Y="${pi/2}"
         prefix="${prefix}top_"
-        parent="${parent}"
+        parent="${prefix}double_sided_shelf"
         scale="${scale}"
     />
-    <joint name="${prefix}double_sided_shelf_left_shelf_joint" type="fixed">
+    <joint name="${prefix}double_sided_shelf_joint" type="fixed">
       <parent link="${parent}" />
-      <child link="${prefix}left_shelf" />
-      <origin rpy="0 0 1.57079632679" xyz="${scale * 4 + x} ${y} ${z}" />
-    </joint>
-    <joint name="${prefix}double_sided_shelf_right_shelf_joint" type="fixed">
-      <parent link="${parent}" />
-      <child link="${prefix}right_shelf" />
-      <origin rpy="0 0 1.57079632679" xyz="${scale * 9 + x} ${y} ${z}" />
-    </joint>
-    <joint name="${prefix}double_sided_shelf_bottom_wall_4x12in_joint" type="fixed">
-      <parent link="${parent}" />
-      <child link="${prefix}bottom_wall_4x12in" />
-      <origin rpy="1.57079632679 0 1.57079632679" xyz="${scale * 4 + x} ${y} ${z}" />
-    </joint>
-    <joint name="${prefix}double_sided_shelf_top_wall_4x12in_joint" type="fixed">
-      <parent link="${parent}" />
-      <child link="${prefix}top_wall_4x12in" />
-      <origin rpy="1.57079632679 0 1.57079632679" xyz="${scale * 4 + x} ${y} ${scale * 4 + z}" />
+      <child link="${prefix}double_sided_shelf" />
+      <origin xyz="${x} ${y} ${z}" rpy="${R} ${P} ${Y}" />
     </joint>
   </xacro:macro>

File: morpheus_teleop/urdf/macros/foam.xacro (robot description, xacro)
@@ -2,5 +2,5 @@
 <robot name="foam" xmlns:xacro="http://www.ros.org/wiki/xacro">
   <xacro:macro name="foam"
-    params="x:=0 y:=0 z:=0 scale:=0.05 prefix parent">
+    params="x:=0 y:=0 z:=0 R:=0 P:=0 Y:=0 scale:=0.05 prefix parent">
     <link name="${prefix}foam">
         <contact>
@@ -34,5 +34,5 @@
       <parent link="${parent}" />
       <child link="${prefix}foam" />
-      <origin xyz="${x} ${y} ${z}" />
+      <origin xyz="${x} ${y} ${z}" rpy="${R} ${P} ${Y}" />
     </joint>
   </xacro:macro>

File: morpheus_teleop/urdf/macros/keyhole.xacro (robot description, xacro)
@@ -5,64 +5,76 @@
   <xacro:include filename="$(find morpheus_teleop)/urdf/macros/wall_4x12in.xacro" />
   <xacro:macro name="keyhole"
-    params="x:=0 y:=0 z:=0 scale:=0.0254 prefix parent">
+    params="x:=0 y:=0 z:=0 R:=0 P:=0 Y:=0 scale:=0.0254 prefix parent">
+    <link name="${prefix}keyhole"/>
     <xacro:shelf
-        prefix="${prefix}"
-        parent="${parent}"
+        x="0"
+        y="0"
+        z="0"
+        R="0"
+        P="0"
+        Y="0"
+        prefix="${prefix}keyhole_shelf_"
+        parent="${prefix}keyhole"
         scale="${scale}"
     />
     <xacro:bar_4in
-        prefix="${prefix}1"
-        parent="${parent}"
+        x="${scale * 4}"
+        y="${scale * 4}"
+        z="${scale * 5}"
+        R="1.57079632679"
+        P="0"
+        Y="0"
+        prefix="${prefix}keyhole_spacer1_"
+        parent="${prefix}keyhole"
         scale="${scale}"
     />
     <xacro:bar_4in
-        prefix="${prefix}2"
-        parent="${parent}"
+        x="${scale * 7}"
+        y="${scale * 4}"
+        z="${scale * 5}"
+        R="1.57079632679"
+        P="0"
+        Y="0"
+        prefix="${prefix}keyhole_spacer2_"
+        parent="${prefix}keyhole"
         scale="${scale}"
     />
     <xacro:bar_4in
-        prefix="${prefix}3"
-        parent="${parent}"
+        x="${scale * 4}"
+        y="${scale * 4}"
+        z="${scale * 6}"
+        R="1.57079632679"
+        P="0"
+        Y="0"
+        prefix="${prefix}keyhole_spacer3_"
+        parent="${prefix}keyhole"
         scale="${scale}"
     />
     <xacro:bar_4in
-        prefix="${prefix}4"
-        parent="${parent}"
+        x="${scale * 7}"
+        y="${scale * 4}"
+        z="${scale * 6}"
+        R="1.57079632679"
+        P="0"
+        Y="0"
+        prefix="${prefix}keyhole_spacer4_"
+        parent="${prefix}keyhole"
         scale="${scale}"
     />
     <xacro:wall_4x12in
-        prefix="${prefix}"
-        parent="${parent}"
+        x="0"
+        y="0"
+        z="${scale * 7}"
+        R="0"
+        P="0"
+        Y="0"
+        prefix="${prefix}keyhole_top_"
+        parent="${prefix}keyhole"
         scale="${scale}"
     />
-    <joint name="${prefix}keyhole_shelf_joint" type="fixed">
+    <joint name="${prefix}keyhole_joint" type="fixed">
       <parent link="${parent}" />
-      <child link="${prefix}shelf" />
-      <origin rpy="0 0 0" xyz="${x} ${y} ${z}" />
-    </joint>
-    <joint name="${prefix}keyhole_1bar_4in_joint" type="fixed">
-      <parent link="${parent}" />
-      <child link="${prefix}1bar_4in" />
-      <origin rpy="1.57079632679 0 0" xyz="${scale * 4 + x} ${scale * 4 + y} ${scale * 5 + z}" />
-    </joint>
-    <joint name="${prefix}keyhole_2bar_4in_joint" type="fixed">
-      <parent link="${parent}" />
-      <child link="${prefix}2bar_4in" />
-      <origin rpy="1.57079632679 0 0" xyz="${scale * 7 + x} ${scale * 4 + y} ${scale * 5 + z}" />
-    </joint>
-    <joint name="${prefix}keyhole_3bar_4in_joint" type="fixed">
-      <parent link="${parent}" />
-      <child link="${prefix}3bar_4in" />
-      <origin rpy="1.57079632679 0 0" xyz="${scale * 4 + x} ${scale * 4 + y} ${scale * 6 + z}" />
-    </joint>
-    <joint name="${prefix}keyhole_4bar_4in_joint" type="fixed">
-      <parent link="${parent}" />
-      <child link="${prefix}4bar_4in" />
-      <origin rpy="1.57079632679 0 0" xyz="${scale * 7 + x} ${scale * 4 + y} ${scale * 6 + z}" />
-    </joint>
-    <joint name="${prefix}keyhole_wall_4x12in_joint" type="fixed">
-      <parent link="${parent}" />
-      <child link="${prefix}wall_4x12in" />
-      <origin rpy="0 0 0" xyz="${x} ${y} ${scale * 7 + z}" />
+      <child link="${prefix}keyhole" />
+      <origin xyz="${x} ${y} ${z}" rpy="${R} ${P} ${Y}" />
     </joint>
   </xacro:macro>

File: morpheus_teleop/urdf/macros/large_tunnel.xacro (robot description, xacro)
@@ -3,44 +3,54 @@
   <xacro:include filename="$(find morpheus_teleop)/urdf/macros/wall_4x12in.xacro" />
   <xacro:macro name="large_tunnel"
-    params="x:=0 y:=0 z:=0 scale:=0.0254 prefix parent">
+    params="x:=0 y:=0 z:=0 R:=0 P:=0 Y:=0 scale:=0.0254 prefix parent">
+    <link name="${prefix}large_tunnel"/>
     <xacro:wall_4x12in
+        x="0"
+        y="0"
+        z="0"
+        R="0"
+        P="0"
+        Y="0"
         prefix="${prefix}bottom"
-        parent="${parent}"
+        parent="${prefix}large_tunnel"
         scale="${scale}"
     />
     <xacro:wall_4x12in
+        x="${scale * 1}"
+        y="${0}"
+        z="${scale * 1}"
+        R="0"
+        P="-1.57079632679"
+        Y="0"
         prefix="${prefix}left"
-        parent="${parent}"
+        parent="${prefix}large_tunnel"
         scale="${scale}"
     />
     <xacro:wall_4x12in
+        x="${scale * 12}"
+        y="${0}"
+        z="${scale * 1}"
+        R="0"
+        P="-1.57079632679"
+        Y="0"
         prefix="${prefix}right"
-        parent="${parent}"
+        parent="${prefix}large_tunnel"
         scale="${scale}"
     />
     <xacro:wall_4x12in
+        x="${0}"
+        y="${0}"
+        z="${scale * 13}"
+        R="0"
+        P="0"
+        Y="0"
         prefix="${prefix}top"
-        parent="${parent}"
+        parent="${prefix}large_tunnel"
         scale="${scale}"
     />
-    <joint name="${prefix}large_tunnel_bottomwall_4x12in_joint" type="fixed">
+    <joint name="${prefix}large_tunnel_joint" type="fixed">
       <parent link="${parent}" />
-      <child link="${prefix}bottomwall_4x12in" />
-      <origin rpy="0 0 0" xyz="${x} ${y} ${z}" />
-    </joint>
-    <joint name="${prefix}large_tunnel_leftwall_4x12in_joint" type="fixed">
-      <parent link="${parent}" />
-      <child link="${prefix}leftwall_4x12in" />
-      <origin rpy="0 -1.57079632679 0" xyz="${scale * 1 + x} ${y} ${scale * 1 + z}" />
-    </joint>
-    <joint name="${prefix}large_tunnel_rightwall_4x12in_joint" type="fixed">
-      <parent link="${parent}" />
-      <child link="${prefix}rightwall_4x12in" />
-      <origin rpy="0 -1.57079632679 0" xyz="${scale * 12 + x} ${y} ${scale * 1 + z}" />
-    </joint>
-    <joint name="${prefix}large_tunnel_topwall_4x12in_joint" type="fixed">
-      <parent link="${parent}" />
-      <child link="${prefix}topwall_4x12in" />
-      <origin rpy="0 0 0" xyz="${x} ${y} ${scale * 13 + z}" />
+      <child link="${prefix}large_tunnel" />
+      <origin xyz="${x} ${y} ${z}" rpy="${R} ${P} ${Y}" />
     </joint>
   </xacro:macro>

File: morpheus_teleop/urdf/macros/shelf.xacro (robot description, xacro)
@@ -4,56 +4,51 @@
   <xacro:include filename="$(find morpheus_teleop)/urdf/macros/bar_4in.xacro" />
   <xacro:macro name="shelf"
-    params="x:=0 y:=0 z:=0 scale:=0.0254 prefix parent">
+    params="x:=0 y:=0 z:=0 R:=0 P:=0 Y:=0 scale:=0.0254 prefix parent">
     <link name="${prefix}shelf"/>
     <xacro:wall_4x12in
+        x="${x}"
+        y="${y}"
+        z="${scale * 4 + z}"
         prefix="${prefix}shelf_"
-        parent="${parent}"
+        parent="${prefix}shelf"
         scale="${scale}"
     />
     <xacro:bar_4in
+        x="${x}"
+        y="${y}"
+        z="${z}"
         prefix="${prefix}shelf_1"
-        parent="${parent}"
+        parent="${prefix}shelf"
         scale="${scale}"
     />
     <xacro:bar_4in
+        x="${scale * 11 + x}"
+        y="${y}"
+        z="${z}"
         prefix="${prefix}shelf_2"
-        parent="${parent}"
+        parent="${prefix}shelf"
         scale="${scale}"
     />
     <xacro:bar_4in
+        x="${x}"
+        y="${scale * 3 + y}"
+        z="${z}"
         prefix="${prefix}shelf_3"
-        parent="${parent}"
+        parent="${prefix}shelf"
         scale="${scale}"
     />
     <xacro:bar_4in
+        x="${scale * 11 + x}"
+        y="${scale * 3 + y}"
+        z="${z}"
         prefix="${prefix}shelf_4"
-        parent="${parent}"
+        parent="${prefix}shelf"
         scale="${scale}"
     />
-    <joint name="${prefix}shelf_wall_4x12in_joint" type="fixed">
-      <parent link="${prefix}shelf" />
-      <child link="${prefix}shelf_wall_4x12in" />
-      <origin xyz="${x} ${y} ${scale * 4 + z}" />
-    </joint>
-    <joint name="${prefix}shelf_leg1_joint" type="fixed">
-      <parent link="${prefix}shelf" />
-      <child link="${prefix}shelf_1bar_4in" />
-      <origin xyz="${x} ${y} ${z}" />
-    </joint>
-    <joint name="${prefix}shelf_leg2_joint" type="fixed">
-      <parent link="${prefix}shelf" />
-      <child link="${prefix}shelf_2bar_4in" />
-      <origin xyz="${scale * 11 + x} ${y} ${z}" />
-    </joint>
-    <joint name="${prefix}shelf_leg3_joint" type="fixed">
-      <parent link="${prefix}shelf" />
-      <child link="${prefix}shelf_3bar_4in" />
-      <origin xyz="${x} ${scale * 3 + y} ${z}" />
-    </joint>
-    <joint name="${prefix}shelf_leg4_joint" type="fixed">
-      <parent link="${prefix}shelf" />
-      <child link="${prefix}shelf_4bar_4in" />
-      <origin xyz="${scale * 11 + x} ${scale * 3 + y} ${z}" />
-    </joint>
+    <joint name="${prefix}shelf_joint" type="fixed">
+        <parent link="${parent}" />
+        <child link="${prefix}shelf" />
+        <origin xyz="${x} ${y} ${z}" rpy="${R} ${P} ${Y}" />
+      </joint>
   </xacro:macro>
 </robot>

File: morpheus_teleop/urdf/macros/table_2x8ft.xacro (robot description, xacro)
@@ -2,5 +2,5 @@
 <robot name="table_2x8ft" xmlns:xacro="http://www.ros.org/wiki/xacro">
   <xacro:macro name="table_2x8ft"
-    params="x:=0 y:=0 z:=0 scale:=0.0254 prefix parent">
+    params="x:=0 y:=0 z:=0 R:=0 P:=0 Y:=0 scale:=0.0254 prefix parent">
     <link name="${prefix}table_2x8ft">
         <inertial>

File: morpheus_teleop/urdf/macros/trees.xacro (robot description, xacro)
@@ -4,44 +4,54 @@
   <xacro:include filename="$(find morpheus_teleop)/urdf/macros/wall_4x12in.xacro" />
   <xacro:macro name="trees"
-    params="x:=0 y:=0 z:=0 scale:=0.0254 prefix parent">
+    params="x:=0 y:=0 z:=0 R:=0 P:=0 Y:=0 scale:=0.0254 prefix parent">
+    <link name="${prefix}trees"/>
     <xacro:wall_4x12in
+        x="0"
+        y="0"
+        z="0"
+        R="0"
+        P="${pi/2}"
+        Y="0"
         prefix="${prefix}"
-        parent="${parent}"
+        parent="${prefix}trees"
         scale="${scale}"
     />
     <xacro:bar_4in
+        x="0"
+        y="0"
+        z="${scale * 1}"
+        R="0"
+        P="0"
+        Y="0"
         prefix="${prefix}1"
-        parent="${parent}"
+        parent="${prefix}trees"
         scale="${scale}"
     />
     <xacro:bar_4in
+        x="${scale * 5.5}"
+        y="0"
+        z="${scale * 1}"
+        R="0"
+        P="0"
+        Y="0"
         prefix="${prefix}2"
-        parent="${parent}"
+        parent="${prefix}trees"
         scale="${scale}"
     />
     <xacro:bar_4in
+        x="${scale * 11}"
+        y="0"
+        z="${scale * 1}"
+        R="0"
+        P="0"
+        Y="0"
         prefix="${prefix}3"
-        parent="${parent}"
+        parent="${prefix}trees"
         scale="${scale}"
     />
-    <joint name="${prefix}trees_wall_4x12in_joint" type="fixed">
+    <joint name="${prefix}trees_joint" type="fixed">
       <parent link="${parent}" />
-      <child link="${prefix}wall_4x12in" />
-      <origin rpy="0 1.57079632679 0" xyz="${x} ${y} ${z}" />
-    </joint>
-    <joint name="${prefix}trees_1bar_4in_joint" type="fixed">
-      <parent link="${parent}" />
-      <child link="${prefix}1bar_4in" />
-      <origin rpy="0 0 0" xyz="${x} ${y} ${scale * 1 + z}" />
-    </joint>
-    <joint name="${prefix}trees_2bar_4in_joint" type="fixed">
-      <parent link="${parent}" />
-      <child link="${prefix}2bar_4in" />
-      <origin rpy="0 0 0" xyz="${scale * 5.5 + x} ${y} ${scale * 1 + z}" />
-    </joint>
-    <joint name="${prefix}trees_3bar_4in_joint" type="fixed">
-      <parent link="${parent}" />
-      <child link="${prefix}3bar_4in" />
-      <origin rpy="0 0 0" xyz="${scale * 11 + x} ${y} ${scale * 1 + z}" />
+      <child link="${prefix}trees"/>
+      <origin xyz="${x} ${y} ${z}" rpy="${R} ${P} ${Y}" />
     </joint>
   </xacro:macro>

File: morpheus_teleop/urdf/macros/tunnel.xacro (robot description, xacro)
@@ -4,44 +4,54 @@
   <xacro:include filename="$(find morpheus_teleop)/urdf/macros/wall_6x12in.xacro" />
   <xacro:macro name="tunnel"
-    params="x:=0 y:=0 z:=0 scale:=0.0254 prefix parent">
+    params="x:=0 y:=0 z:=0 R:=0 P:=0 Y:=0 scale:=0.0254 prefix parent">
+    <link name="${prefix}tunnel"/>
     <xacro:wall_6x12in
-        prefix="${prefix}bottom"
-        parent="${parent}"
+        x="0"
+        y="0"
+        z="0"
+        R="0"
+        P="0"
+        Y="1.57079632679"
+        prefix="${prefix}tunnel_bottom_"
+        parent="${prefix}tunnel"
         scale="${scale}"
     />
     <xacro:wall_4x12in
-        prefix="${prefix}left"
-        parent="${parent}"
+        x="0"
+        y="0"
+        z="${scale * 1}"
+        R="1.57079632679"
+        P="1.57079632679"
+        Y="0"
+        prefix="${prefix}tunnel_left_"
+        parent="${prefix}tunnel"
         scale="${scale}"
     />
     <xacro:wall_4x12in
-        prefix="${prefix}right"
-        parent="${parent}"
+        x="${scale * 5}"
+        y="0"
+        z="${scale * 1}"
+        R="1.57079632679"
+        P="1.57079632679"
+        Y="0"
+        prefix="${prefix}tunnel_right_"
+        parent="${prefix}tunnel"
         scale="${scale}"
     />
     <xacro:wall_6x12in
-        prefix="${prefix}top"
-        parent="${parent}"
+        x="0"
+        y="0"
+        z="${scale * 5}"
+        R="0"
+        P="0"
+        Y="1.57079632679"
+        prefix="${prefix}tunnel_top_"
+        parent="${prefix}tunnel"
         scale="${scale}"
     />
-    <joint name="${prefix}tunnel_bottomwall_6x12in_joint" type="fixed">
+    <joint name="${prefix}tunnel_joint" type="fixed">
       <parent link="${parent}" />
-      <child link="${prefix}bottomwall_4x12in" />
-      <origin rpy="0 0 1.57079632679" xyz="${x} ${y} ${z}" />
-    </joint>
-    <joint name="${prefix}tunnel_leftwall_4x12in_joint" type="fixed">
-      <parent link="${parent}" />
-      <child link="${prefix}leftwall_4x12in" />
-      <origin rpy="1.57079632679 1.57079632679 0" xyz="${x} ${y} ${scale * 1 + z}" />
-    </joint>
-    <joint name="${prefix}tunnel_rightwall_4x12in_joint" type="fixed">
-      <parent link="${parent}" />
-      <child link="${prefix}rightwall_4x12in" />
-      <origin rpy="1.57079632679 1.57079632679 0" xyz="${scale * 5 + x} ${y} ${scale * 1 + z}" />
-    </joint>
-    <joint name="${prefix}tunnel_topwall_6x12in_joint" type="fixed">
-      <parent link="${parent}" />
-      <child link="${prefix}topwall_4x12in" />
-      <origin rpy="0 0 1.57079632679" xyz="${x} ${y} ${scale * 5 + z}" />
+      <child link="${prefix}tunnel"/>
+      <origin xyz="${x} ${y} ${z}" rpy="${R} ${P} ${Y}" />
     </joint>
   </xacro:macro>
