Commit message: Object spawner fixes, obstacle refactoring

File: morpheus_teleop/urdf/macros/wall_4x12in.xacro (robot description, xacro)
@@ -2,5 +2,5 @@
 <robot name="wall_4x12in" xmlns:xacro="http://www.ros.org/wiki/xacro">
   <xacro:macro name="wall_4x12in"
-    params="x:=0 y:=0 z:=0 scale:=0.0254 prefix parent">
+    params="x:=0 y:=0 z:=0 R:=0 P:=0 Y:=0 scale:=0.0254 prefix parent">
     <link name="${prefix}wall_4x12in">
         <contact>
@@ -31,4 +31,9 @@
         </collision>
     </link>
+    <joint name="${prefix}wall_4x12in_joint" type="fixed">
+        <parent link="${parent}" />
+        <child link="${prefix}wall_4x12in" />
+        <origin xyz="${x} ${y} ${z}" rpy="${R} ${P} ${Y}" />
+    </joint>
   </xacro:macro>
 </robot>

File: morpheus_teleop/urdf/macros/wall_6x12in.xacro (robot description, xacro)
@@ -31,4 +31,9 @@
         </collision>
     </link>
+    <joint name="${prefix}wall_6x12in_joint" type="fixed">
+        <parent link="${parent}" />
+        <child link="${prefix}wall_6x12in" />
+        <origin xyz="${x} ${y} ${z}" rpy="${R} ${P} ${Y}" />
+    </joint>
   </xacro:macro>
 </robot>

File: morpheus_teleop/urdf/scenes/bar_12in_scene.xacro (robot description, xacro)
@@ -1,11 +1,12 @@
 <?xml version="1.0"?>
-<robot xmlns:xacro="http://www.ros.org/wiki/xacro" name="block_scene">
+<robot xmlns:xacro="http://www.ros.org/wiki/xacro" name="bar_12in_scene">
+    <link name="base_link" />
     <xacro:include filename="$(find morpheus_teleop)/urdf/macros/bar_12in.xacro" />
     <xacro:bar_12in
         prefix=""
-        parent="world"
-        x="-0.5"
-        y="1.0"
-        z="0.74295"
+        parent="base_link"
+        x="-0.0127"
+        y="-0.1528"
+        z="-0.0127"
         scale="0.0254"
     />

File: morpheus_teleop/urdf/scenes/block_scene.xacro (robot description, xacro)
@@ -1,11 +1,12 @@
 <?xml version="1.0"?>
 <robot xmlns:xacro="http://www.ros.org/wiki/xacro" name="block_scene">
+    <link name="base_link" />
     <xacro:include filename="$(find morpheus_teleop)/urdf/macros/block.xacro" />
     <xacro:block
         prefix=""
-        parent="world"
-        x="-0.5"
-        y="1.0"
-        z="0.74295"
+        parent="base_link"
+        x="0.0"
+        y="0.0"
+        z="0.0"
         scale="0.0254"
     />
