Commit message: Node 2 scene tweaks

File: morpheus_teleop/urdf/macros/node2.xacro (robot description, xacro)
@@ -51,5 +51,5 @@
         <parent link="${parent}" />
         <child link="${prefix}node2" />
-        <origin xyz="${x} ${y} ${z}" rpy="${R} ${P} ${Y + pi}" />
+        <origin xyz="${x} ${y} ${z}" rpy="${R} ${P} ${Y + 3*pi/2}" />
     </joint>
     <joint name="${prefix}PMA3_joint" type="fixed">

File: morpheus_teleop/urdf/macros/node2_table.xacro (robot description, xacro)
@@ -16,5 +16,5 @@
         prefix=""
         parent="world"
-        x="${x + (0.0254 * 63)}"
+        x="${x + (0.0254 * 48)}"
         y="${y + (0.0254 * 14.5)}"
         z="${z + (0.0254 * 34.75) + (0.0254 * 21)}"

File: morpheus_teleop/urdf/scenes/b_bot_node2_scene.xacro (robot description, xacro)
@@ -6,5 +6,5 @@
         prefix=""
         parent="world"
-        x="${0.0254 * (-62)}"
+        x="${0.0254 * (-48)}"
         y="${0.0254 * 8.5}"
         z="0"
