Commit message: Trossen launch files in progress

File: morpheus_teleop/urdf/macros/trossen_macro.xacro (robot description, xacro)
@@ -1,25 +1,14 @@
 <?xml version="1.0"?>
 <robot xmlns:xacro="http://www.ros.org/wiki/xacro" name="trossen">
-    <xacro:macro name="vx300s">
-        <xacro:include filename="$(find interbotix_xsarm_descriptions)/urdf/vx300s.urdf.xacro" />
-        <link name="world"/>
-        <joint name="fixed" type="fixed">
-            <parent link="${parent}"/>
-            <child link="$(arg robot_name)/$(arg base_link_frame)"/>
-        </joint>
-    </xacro:macro>
+    <xacro:include filename="$(find morpheus_teleop)/urdf/macros/vx300s_macro.xacro" />
     <xacro:macro name="trossen"
         params="
         prefix
         parent
-        transmission_hw_interface:=hardware_interface/PositionJointInterface
-        joint_limits_parameters_file:='$(find interbotix_xsarm_moveit)/config/joint_limits/6dof_joint_limits.yaml'
         *origin">
         <xacro:vx300s
             prefix="${prefix}"
             parent="${parent}"
-            tcp_offset="0.223"
-            joint_limits_parameters_file="${joint_limits_parameters_file}"
-            transmission_hw_interface="${transmission_hw_interface}"
+            tcp_offset="0.163"
         >
             <origin xyz="0 0 0" rpy="0 0 0" />

File: morpheus_teleop/urdf/scenes/trossen_node2_scene.xacro (robot description, xacro)
@@ -1,4 +1,4 @@
 <?xml version="1.0"?>
-<robot xmlns:xacro="http://www.ros.org/wiki/xacro" name="b_bot_node2_scene">
+<robot xmlns:xacro="http://www.ros.org/wiki/xacro" name="trossen_node2_scene">
     <xacro:include filename="$(find morpheus_teleop)/urdf/scenes/trossen_scene.xacro" />
     <xacro:include filename="$(find morpheus_teleop)/urdf/macros/node2_table.xacro" />

File: morpheus_teleop/urdf/scenes/trossen_scene.xacro (robot description, xacro)
@@ -1,9 +1,6 @@
 <?xml version="1.0"?>
-<robot xmlns:xacro="http://www.ros.org/wiki/xacro" name="b_bot_scene">
-    <xacro:arg name="joint_limits_parameters_file"
-        default="$(find interbotix_xsarm_moveit)/config/joint_limits/6dof_joint_limits.yaml" />
-    <xacro:arg name="transmission_hw_interface" default="hardware_interface/PositionJointInterface" />
+<robot xmlns:xacro="http://www.ros.org/wiki/xacro" name="trossen_scene">
     <xacro:include filename="$(find homestri_description)/urdf/macros/simple_pedestal_macro.xacro" />
-    <xacro:include filename="$(find homestri_description)/urdf/macros/trossen_macro.xacro" />
+    <xacro:include filename="$(find morpheus_teleop)/urdf/macros/trossen_macro.xacro" />
     <xacro:simple_pedestal
         prefix=""
@@ -12,13 +9,10 @@
         radius="0.15"
     />
-    <xacro:b_bot
+    <xacro:trossen
         prefix=""
         parent="pedestal"
-        transmission_hw_interface="$(arg transmission_hw_interface)"
-        joint_limits_parameters_file="$(arg joint_limits_parameters_file)"
     >
         <origin xyz="0 0 0" rpy="0 0 0" />
-    </xacro:b_bot>
-    <link name="world" />
+    </xacro:trossen>
     <gazebo>
         <plugin name="ros_control" filename="libgazebo_ros_control.so">
