Commit message: Keyboard simulation of joystick enabled. Obstacles and analysis module in progress

File: morpheus_teleop/urdf/macros/Test_Block_1.xacro (robot description, xacro)
@@ -1,7 +1,7 @@
 <?xml version="1.0"?>
-<robot name="Test_Block_1" xmlns:xacro="http://www.ros.org/wiki/xacro">
-  <xacro:macro name="Test_Block_1"
+<robot name="test_block_1" xmlns:xacro="http://www.ros.org/wiki/xacro">
+  <xacro:macro name="test_block_1"
     params="x:=0 y:=0 z:=0 scale:=0.001 prefix parent">
-    <link name="${prefix}Test_Block_1">
+    <link name="${prefix}test_block_1">
         <contact>
             <lateral_friction value="1.0"/>
@@ -18,5 +18,5 @@
             <origin rpy="0 0 0" xyz="0 0 0"/>
             <geometry>
-                <mesh filename="package://morpheus_teleop/meshes/components/visual/Test_Block_1.stl" scale="${scale} ${scale} ${scale}"/>
+                <mesh filename="package://morpheus_teleop/meshes/components/visual/test_block_1.stl" scale="${scale} ${scale} ${scale}"/>
             </geometry>
             <material name="grey">
@@ -27,11 +27,11 @@
             <origin rpy="0 0 0" xyz="0 0 0" />
             <geometry>
-                <mesh filename="package://morpheus_teleop/meshes/components/collision/Test_Block_1.stl" scale="${scale} ${scale} ${scale}"/>
+                <mesh filename="package://morpheus_teleop/meshes/components/collision/test_block_1.stl" scale="${scale} ${scale} ${scale}"/>
             </geometry>
         </collision>
     </link>
-    <joint name="${prefix}Test_Block_1_joint" type="fixed">
+    <joint name="${prefix}test_block_1_joint" type="fixed">
       <parent link="${parent}" />
-      <child link="${prefix}Test_Block_1" />
+      <child link="${prefix}test_block_1" />
       <origin xyz="${x} ${y} ${z}" />
     </joint>

File: morpheus_teleop/urdf/scenes/test_wall_1_scene.xacro (robot description, xacro)
@@ -1,4 +1,4 @@
 <?xml version="1.0"?>
-<robot xmlns:xacro="http://www.ros.org/wiki/xacro" name="test_scene">
+<robot xmlns:xacro="http://www.ros.org/wiki/xacro" name="test_wall_1_scene">
     <xacro:include filename="$(find morpheus_teleop)/urdf/scenes/a_bot_scene.xacro" />
     <xacro:include filename="$(find morpheus_teleop)/urdf/macros/test_wall_1.xacro" />
