Commit message: Obstacles rewritten to be assemblies of sub-macros

File: morpheus_teleop/urdf/macros/Test_Block_1.xacro (robot description, xacro)
@@ -11,5 +11,5 @@
         </contact>
         <inertial>
-            <origin rpy="0 0 0" xyz="0.0 0.0 0.03"/>
+            <origin rpy="0 0 0" xyz="0.0 0.0 0.0"/>
             <mass value="2"/>
             <inertia ixx="1.0" ixy="0" ixz="0" iyy="1" iyz="0" izz="1"/>

File: morpheus_teleop/urdf/macros/block.xacro (robot description, xacro)
@@ -1,7 +1,7 @@
 <?xml version="1.0"?>
-<robot name="wall" xmlns:xacro="http://www.ros.org/wiki/xacro">
-  <xacro:macro name="wall"
-    params="x:=0 y:=0 z:=0 scale:=0.05 prefix parent">
-    <link name="${prefix}wall">
+<robot name="block" xmlns:xacro="http://www.ros.org/wiki/xacro">
+  <xacro:macro name="block"
+    params="x:=0 y:=0 z:=0 scale:=0.0254 prefix parent">
+    <link name="${prefix}block">
         <contact>
             <lateral_friction value="1.0"/>
@@ -11,5 +11,5 @@
         </contact>
         <inertial>
-            <origin rpy="0 0 0" xyz="0.0 0.0 0.0"/>
+            <origin rpy="0 0 0" xyz="0.0 0.0 0.0125"/>
             <mass value="1"/>
             <inertia ixx="1" ixy="0" ixz="0" iyy="1" iyz="0" izz="1"/>
@@ -18,5 +18,5 @@
             <origin rpy="1.57079632679 0 0" xyz="0 0 0"/>
             <geometry>
-                <mesh filename="package://morpheus_teleop/meshes/components/visual/wall.obj" scale="${scale} ${scale} ${scale}"/>
+                <mesh filename="package://morpheus_teleop/meshes/components/visual/block.obj" scale="${scale} ${scale} ${scale}"/>
             </geometry>
             <material name="grey">
@@ -27,13 +27,8 @@
             <origin rpy="1.57079632679 0 0" xyz="0 0 0" />
             <geometry>
-                <mesh filename="package://morpheus_teleop/meshes/components/collision/wall.obj" scale="${scale} ${scale} ${scale}"/>
+                <mesh filename="package://morpheus_teleop/meshes/components/collision/block.obj" scale="${scale} ${scale} ${scale}"/>
             </geometry>
         </collision>
     </link>
-    <joint name="${prefix}wall_joint" type="fixed">
-      <parent link="${parent}" />
-      <child link="${prefix}wall" />
-      <origin xyz="${x} ${y} ${z}" />
-    </joint>
   </xacro:macro>
 </robot>

File: morpheus_teleop/urdf/macros/double_sided_shelf.xacro (robot description, xacro)
@@ -1,38 +1,47 @@
 <?xml version="1.0"?>
 <robot name="double_sided_shelf" xmlns:xacro="http://www.ros.org/wiki/xacro">
+  <xacro:include filename="$(find morpheus_teleop)/urdf/macros/shelf.xacro" />
+  <xacro:include filename="$(find morpheus_teleop)/urdf/macros/wall_4x12in.xacro" />
   <xacro:macro name="double_sided_shelf"
-    params="x:=0 y:=0 z:=0 scale:=0.05 prefix parent">
-    <link name="${prefix}double_sided_shelf">
-        <contact>
-            <lateral_friction value="1.0"/>
-            <rolling_friction value="0.0"/>
-            <contact_cfm value="0.0"/>
-            <contact_erp value="1.0"/>
-        </contact>
-        <inertial>
-            <origin rpy="0 0 0" xyz="0.0 0.0 0.03"/>
-            <mass value="1"/>
-            <inertia ixx="1" ixy="0" ixz="0" iyy="1" iyz="0" izz="1"/>
-        </inertial>
-        <visual>
-            <origin rpy="1.57079632679 0 0" xyz="0 0 0"/>
-            <geometry>
-                <mesh filename="package://morpheus_teleop/meshes/components/visual/double_sided_shelf.obj" scale="${scale} ${scale} ${scale}"/>
-            </geometry>
-            <material name="grey">
-                <color rgba="0.3 0.3 0.3 1" />
-            </material>
-        </visual>
-        <collision>
-            <origin rpy="1.57079632679 0 0" xyz="0 0 0" />
-            <geometry>
-                <mesh filename="package://morpheus_teleop/meshes/components/collision/double_sided_shelf.obj" scale="${scale} ${scale} ${scale}"/>
-            </geometry>
-        </collision>
-    </link>
-    <joint name="${prefix}double_sided_shelf_joint" type="fixed">
+    params="x:=0 y:=0 z:=0 scale:=0.0254 prefix parent">
+    <xacro:shelf
+        prefix="${prefix}left_"
+        parent="${parent}"
+        scale="${scale}"
+    />
+    <xacro:shelf
+        prefix="${prefix}right_"
+        parent="${parent}"
+        scale="${scale}"
+    />
+    <xacro:wall_4x12in
+        prefix="${prefix}bottom_"
+        parent="${parent}"
+        scale="${scale}"
+    />
+    <xacro:wall_4x12in
+        prefix="${prefix}top_"
+        parent="${parent}"
+        scale="${scale}"
+    />
+    <joint name="${prefix}double_sided_shelf_left_shelf_joint" type="fixed">
       <parent link="${parent}" />
-      <child link="${prefix}double_sided_shelf" />
-      <origin xyz="${x} ${y} ${z}" />
+      <child link="${prefix}left_shelf" />
+      <origin rpy="0 0 1.57079632679" xyz="${scale * 4 + x} ${y} ${z}" />
+    </joint>
+    <joint name="${prefix}double_sided_shelf_right_shelf_joint" type="fixed">
+      <parent link="${parent}" />
+      <child link="${prefix}right_shelf" />
+      <origin rpy="0 0 1.57079632679" xyz="${scale * 9 + x} ${y} ${z}" />
+    </joint>
+    <joint name="${prefix}double_sided_shelf_bottom_wall_4x12in_joint" type="fixed">
+      <parent link="${parent}" />
+      <child link="${prefix}bottom_wall_4x12in" />
+      <origin rpy="1.57079632679 0 1.57079632679" xyz="${scale * 4 + x} ${y} ${z}" />
+    </joint>
+    <joint name="${prefix}double_sided_shelf_top_wall_4x12in_joint" type="fixed">
+      <parent link="${parent}" />
+      <child link="${prefix}top_wall_4x12in" />
+      <origin rpy="1.57079632679 0 1.57079632679" xyz="${scale * 4 + x} ${y} ${scale * 4 + z}" />
     </joint>
   </xacro:macro>

File: morpheus_teleop/urdf/macros/double_sided_shelf_solid.xacro (robot description, xacro)
@@ -1,7 +1,7 @@
 <?xml version="1.0"?>
-<robot name="wall" xmlns:xacro="http://www.ros.org/wiki/xacro">
-  <xacro:macro name="wall"
-    params="x:=0 y:=0 z:=0 scale:=0.05 prefix parent">
-    <link name="${prefix}wall">
+<robot name="double_sided_shelf" xmlns:xacro="http://www.ros.org/wiki/xacro">
+  <xacro:macro name="double_sided_shelf"
+    params="x:=0 y:=0 z:=0 scale:=0.0254 prefix parent">
+    <link concave="yes" name="${prefix}double_sided_shelf">
         <contact>
             <lateral_friction value="1.0"/>
@@ -18,5 +18,5 @@
             <origin rpy="1.57079632679 0 0" xyz="0 0 0"/>
             <geometry>
-                <mesh filename="package://morpheus_teleop/meshes/components/visual/wall.obj" scale="${scale} ${scale} ${scale}"/>
+                <mesh filename="package://morpheus_teleop/meshes/components/visual/double_sided_shelf.obj" scale="${scale} ${scale} ${scale}"/>
             </geometry>
             <material name="grey">
@@ -24,14 +24,14 @@
             </material>
         </visual>
-        <collision>
+        <collision concave="yes">
             <origin rpy="1.57079632679 0 0" xyz="0 0 0" />
             <geometry>
-                <mesh filename="package://morpheus_teleop/meshes/components/collision/wall.obj" scale="${scale} ${scale} ${scale}"/>
+                <mesh filename="package://morpheus_teleop/meshes/components/collision/double_sided_shelf.obj" scale="${scale} ${scale} ${scale}"/>
             </geometry>
         </collision>
     </link>
-    <joint name="${prefix}wall_joint" type="fixed">
+    <joint name="${prefix}double_sided_shelf_joint" type="fixed">
       <parent link="${parent}" />
-      <child link="${prefix}wall" />
+      <child link="${prefix}double_sided_shelf" />
       <origin xyz="${x} ${y} ${z}" />
     </joint>

File: morpheus_teleop/urdf/macros/foam.xacro (robot description, xacro)
@@ -11,5 +11,5 @@
         </contact>
         <inertial>
-            <origin rpy="0 0 0" xyz="0.0 0.0 0.03"/>
+            <origin rpy="0 0 0" xyz="0.0 0.0 0.0"/>
             <mass value="1"/>
             <inertia ixx="1" ixy="0" ixz="0" iyy="1" iyz="0" izz="1"/>

File: morpheus_teleop/urdf/macros/keyhole_original.xacro (robot description, xacro)
@@ -1,7 +1,7 @@
 <?xml version="1.0"?>
-<robot name="wall" xmlns:xacro="http://www.ros.org/wiki/xacro">
-  <xacro:macro name="wall"
-    params="x:=0 y:=0 z:=0 scale:=0.05 prefix parent">
-    <link name="${prefix}wall">
+<robot name="keyhole" xmlns:xacro="http://www.ros.org/wiki/xacro">
+  <xacro:macro name="keyhole"
+    params="x:=0 y:=0 z:=0 scale:=0.0254 prefix parent">
+    <link name="${prefix}keyhole">
         <contact>
             <lateral_friction value="1.0"/>
@@ -18,5 +18,5 @@
             <origin rpy="1.57079632679 0 0" xyz="0 0 0"/>
             <geometry>
-                <mesh filename="package://morpheus_teleop/meshes/components/visual/wall.obj" scale="${scale} ${scale} ${scale}"/>
+                <mesh filename="package://morpheus_teleop/meshes/components/visual/keyhole.obj" scale="${scale} ${scale} ${scale}"/>
             </geometry>
             <material name="grey">
@@ -27,11 +27,11 @@
             <origin rpy="1.57079632679 0 0" xyz="0 0 0" />
             <geometry>
-                <mesh filename="package://morpheus_teleop/meshes/components/collision/wall.obj" scale="${scale} ${scale} ${scale}"/>
+                <mesh filename="package://morpheus_teleop/meshes/components/collision/keyhole.obj" scale="${scale} ${scale} ${scale}"/>
             </geometry>
         </collision>
     </link>
-    <joint name="${prefix}wall_joint" type="fixed">
+    <joint name="${prefix}keyhole_joint" type="fixed">
       <parent link="${parent}" />
-      <child link="${prefix}wall" />
+      <child link="${prefix}keyhole" />
       <origin xyz="${x} ${y} ${z}" />
     </joint>

File: morpheus_teleop/urdf/macros/large_tunnel_original.xacro (robot description, xacro)
@@ -1,7 +1,7 @@
 <?xml version="1.0"?>
-<robot name="wall" xmlns:xacro="http://www.ros.org/wiki/xacro">
-  <xacro:macro name="wall"
-    params="x:=0 y:=0 z:=0 scale:=0.05 prefix parent">
-    <link name="${prefix}wall">
+<robot name="large_tunnel" xmlns:xacro="http://www.ros.org/wiki/xacro">
+  <xacro:macro name="large_tunnel"
+    params="x:=0 y:=0 z:=0 scale:=0.0254 prefix parent">
+    <link name="${prefix}large_tunnel">
         <contact>
             <lateral_friction value="1.0"/>
@@ -18,5 +18,5 @@
             <origin rpy="1.57079632679 0 0" xyz="0 0 0"/>
             <geometry>
-                <mesh filename="package://morpheus_teleop/meshes/components/visual/wall.obj" scale="${scale} ${scale} ${scale}"/>
+                <mesh filename="package://morpheus_teleop/meshes/components/visual/large_tunnel.obj" scale="${scale} ${scale} ${scale}"/>
             </geometry>
             <material name="grey">
@@ -27,11 +27,11 @@
             <origin rpy="1.57079632679 0 0" xyz="0 0 0" />
             <geometry>
-                <mesh filename="package://morpheus_teleop/meshes/components/collision/wall.obj" scale="${scale} ${scale} ${scale}"/>
+                <mesh filename="package://morpheus_teleop/meshes/components/collision/large_tunnel.obj" scale="${scale} ${scale} ${scale}"/>
             </geometry>
         </collision>
     </link>
-    <joint name="${prefix}wall_joint" type="fixed">
+    <joint name="${prefix}large_tunnel_joint" type="fixed">
       <parent link="${parent}" />
-      <child link="${prefix}wall" />
+      <child link="${prefix}large_tunnel" />
       <origin xyz="${x} ${y} ${z}" />
     </joint>

File: morpheus_teleop/urdf/macros/table_2x8ft.xacro (robot description, xacro)
@@ -2,19 +2,13 @@
 <robot name="table_2x8ft" xmlns:xacro="http://www.ros.org/wiki/xacro">
   <xacro:macro name="table_2x8ft"
-    params="x:=0 y:=0 z:=0 scale:=0.05 prefix parent">
+    params="x:=0 y:=0 z:=0 scale:=0.0254 prefix parent">
     <link name="${prefix}table_2x8ft">
-        <contact>
-            <lateral_friction value="1.0"/>
-            <rolling_friction value="0.0"/>
-            <contact_cfm value="0.0"/>
-            <contact_erp value="1.0"/>
-        </contact>
         <inertial>
-            <origin rpy="0 0 0" xyz="0.0 0.0 0.03"/>
+            <origin rpy="0 0 0" xyz="0.0 0.0 0.0"/>
             <mass value="1"/>
             <inertia ixx="1" ixy="0" ixz="0" iyy="1" iyz="0" izz="1"/>
         </inertial>
         <visual>
-            <origin rpy="1.57079632679 0 0" xyz="0 0 0"/>
+            <origin rpy="-1.57079632679 0 0" xyz="0 0 ${-scale * 1}"/>
             <geometry>
                 <mesh filename="package://morpheus_teleop/meshes/components/visual/table_2x8ft.obj" scale="${scale} ${scale} ${scale}"/>
@@ -25,5 +19,5 @@
         </visual>
         <collision>
-            <origin rpy="1.57079632679 0 0" xyz="0 0 0" />
+            <origin rpy="-1.57079632679 0 0" xyz="0 0 ${-scale * 1}" />
             <geometry>
                 <mesh filename="package://morpheus_teleop/meshes/components/collision/table_2x8ft.obj" scale="${scale} ${scale} ${scale}"/>

File: morpheus_teleop/urdf/macros/teapot.xacro (robot description, xacro)
@@ -11,5 +11,5 @@
         </contact>
         <inertial>
-            <origin rpy="0 0 0" xyz="0.0 0.0 0.03"/>
+            <origin rpy="0 0 0" xyz="0.0 0.0 0.0"/>
             <mass value="2"/>
             <inertia ixx="1.5" ixy="0" ixz="0" iyy="2" iyz="0" izz="2"/>
@@ -24,5 +24,5 @@
             </material>
         </visual>
-        <collision>
+        <collision concave="yes">
             <origin rpy="1.57079632679 0 0" xyz="0 0 0" />
             <geometry>

File: morpheus_teleop/urdf/macros/test_wall_1.xacro (robot description, xacro)
@@ -11,5 +11,5 @@
         </contact>
         <inertial>
-            <origin rpy="0 0 0" xyz="0.0 0.0 0.03"/>
+            <origin rpy="0 0 0" xyz="0.0 0.0 0.0"/>
             <mass value="1"/>
             <inertia ixx="1" ixy="0" ixz="0" iyy="1" iyz="0" izz="1"/>

File: morpheus_teleop/urdf/macros/trees_original.xacro (robot description, xacro)
@@ -1,7 +1,7 @@
 <?xml version="1.0"?>
-<robot name="wall" xmlns:xacro="http://www.ros.org/wiki/xacro">
-  <xacro:macro name="wall"
-    params="x:=0 y:=0 z:=0 scale:=0.05 prefix parent">
-    <link name="${prefix}wall">
+<robot name="trees" xmlns:xacro="http://www.ros.org/wiki/xacro">
+  <xacro:macro name="trees"
+    params="x:=0 y:=0 z:=0 scale:=0.0254 prefix parent">
+    <link concave="yes" name="${prefix}trees">
         <contact>
             <lateral_friction value="1.0"/>
@@ -12,5 +12,5 @@
         <inertial>
             <origin rpy="0 0 0" xyz="0.0 0.0 0.0"/>
-            <mass value="1"/>
+            <mass value="0.0"/>
             <inertia ixx="1" ixy="0" ixz="0" iyy="1" iyz="0" izz="1"/>
         </inertial>
@@ -18,5 +18,5 @@
             <origin rpy="1.57079632679 0 0" xyz="0 0 0"/>
             <geometry>
-                <mesh filename="package://morpheus_teleop/meshes/components/visual/wall.obj" scale="${scale} ${scale} ${scale}"/>
+                <mesh filename="package://morpheus_teleop/meshes/components/visual/trees.obj" scale="${scale} ${scale} ${scale}"/>
             </geometry>
             <material name="grey">
@@ -24,14 +24,14 @@
             </material>
         </visual>
-        <collision>
+        <collision concave="yes">
             <origin rpy="1.57079632679 0 0" xyz="0 0 0" />
             <geometry>
-                <mesh filename="package://morpheus_teleop/meshes/components/collision/wall.obj" scale="${scale} ${scale} ${scale}"/>
+                <mesh filename="package://morpheus_teleop/meshes/components/collision/trees.obj" scale="${scale} ${scale} ${scale}"/>
             </geometry>
         </collision>
     </link>
-    <joint name="${prefix}wall_joint" type="fixed">
+    <joint name="${prefix}trees_joint" type="fixed">
       <parent link="${parent}" />
-      <child link="${prefix}wall" />
+      <child link="${prefix}trees" />
       <origin xyz="${x} ${y} ${z}" />
     </joint>

File: morpheus_teleop/urdf/macros/tunnel_original.xacro (robot description, xacro)
@@ -1,7 +1,7 @@
 <?xml version="1.0"?>
-<robot name="wall" xmlns:xacro="http://www.ros.org/wiki/xacro">
-  <xacro:macro name="wall"
-    params="x:=0 y:=0 z:=0 scale:=0.05 prefix parent">
-    <link name="${prefix}wall">
+<robot name="tunnel" xmlns:xacro="http://www.ros.org/wiki/xacro">
+  <xacro:macro name="tunnel"
+    params="x:=0 y:=0 z:=0 scale:=0.0254 prefix parent">
+    <link concave="yes" name="${prefix}tunnel">
         <contact>
             <lateral_friction value="1.0"/>
@@ -12,5 +12,5 @@
         <inertial>
             <origin rpy="0 0 0" xyz="0.0 0.0 0.0"/>
-            <mass value="1"/>
+            <mass value="0.0"/>
             <inertia ixx="1" ixy="0" ixz="0" iyy="1" iyz="0" izz="1"/>
         </inertial>
@@ -18,5 +18,5 @@
             <origin rpy="1.57079632679 0 0" xyz="0 0 0"/>
             <geometry>
-                <mesh filename="package://morpheus_teleop/meshes/components/visual/wall.obj" scale="${scale} ${scale} ${scale}"/>
+                <mesh filename="package://morpheus_teleop/meshes/components/visual/tunnel.obj" scale="${scale} ${scale} ${scale}"/>
             </geometry>
             <material name="grey">
@@ -24,14 +24,14 @@
             </material>
         </visual>
-        <collision>
+        <collision concave="yes">
             <origin rpy="1.57079632679 0 0" xyz="0 0 0" />
             <geometry>
-                <mesh filename="package://morpheus_teleop/meshes/components/collision/wall.obj" scale="${scale} ${scale} ${scale}"/>
+                <mesh filename="package://morpheus_teleop/meshes/components/collision/tunnel.obj" scale="${scale} ${scale} ${scale}"/>
             </geometry>
         </collision>
     </link>
-    <joint name="${prefix}wall_joint" type="fixed">
+    <joint name="${prefix}tunnel_joint" type="fixed">
       <parent link="${parent}" />
-      <child link="${prefix}wall" />
+      <child link="${prefix}tunnel" />
       <origin xyz="${x} ${y} ${z}" />
     </joint>

File: morpheus_teleop/urdf/macros/wall_4x12in.xacro (robot description, xacro)
@@ -1,7 +1,7 @@
 <?xml version="1.0"?>
-<robot name="wall" xmlns:xacro="http://www.ros.org/wiki/xacro">
-  <xacro:macro name="wall"
-    params="x:=0 y:=0 z:=0 scale:=0.05 prefix parent">
-    <link name="${prefix}wall">
+<robot name="wall_4x12in" xmlns:xacro="http://www.ros.org/wiki/xacro">
+  <xacro:macro name="wall_4x12in"
+    params="x:=0 y:=0 z:=0 scale:=0.0254 prefix parent">
+    <link name="${prefix}wall_4x12in">
         <contact>
             <lateral_friction value="1.0"/>
@@ -16,7 +16,7 @@
         </inertial>
         <visual>
-            <origin rpy="1.57079632679 0 0" xyz="0 0 0"/>
+            <origin rpy="0 0 1.57079632679" xyz="${scale * 12} 0.0 0.0"/>
             <geometry>
-                <mesh filename="package://morpheus_teleop/meshes/components/visual/wall.obj" scale="${scale} ${scale} ${scale}"/>
+                <mesh filename="package://morpheus_teleop/meshes/components/visual/wall_4x12in.obj" scale="${scale} ${scale} ${scale}"/>
             </geometry>
             <material name="grey">
@@ -25,15 +25,10 @@
         </visual>
         <collision>
-            <origin rpy="1.57079632679 0 0" xyz="0 0 0" />
+            <origin rpy="0 0 1.57079632679" xyz="${scale * 12} 0.0 0.0"/>
             <geometry>
-                <mesh filename="package://morpheus_teleop/meshes/components/collision/wall.obj" scale="${scale} ${scale} ${scale}"/>
+                <mesh filename="package://morpheus_teleop/meshes/components/collision/wall_4x12in.obj" scale="${scale} ${scale} ${scale}"/>
             </geometry>
         </collision>
     </link>
-    <joint name="${prefix}wall_joint" type="fixed">
-      <parent link="${parent}" />
-      <child link="${prefix}wall" />
-      <origin xyz="${x} ${y} ${z}" />
-    </joint>
   </xacro:macro>
 </robot>

File: morpheus_teleop/urdf/scenes/a_bot_double_level_shelf_scene.xacro (robot description, xacro)
@@ -1,4 +1,4 @@
 <?xml version="1.0"?>
-<robot xmlns:xacro="http://www.ros.org/wiki/xacro" name="a_bot_double_sided_shelf_scene">
+<robot xmlns:xacro="http://www.ros.org/wiki/xacro" name="a_bot_double_level_shelf_scene">
     <xacro:include filename="$(find morpheus_teleop)/urdf/scenes/a_bot_scene.xacro" />
     <xacro:include filename="$(find morpheus_teleop)/urdf/macros/table_2x8ft.xacro" />
@@ -6,16 +6,16 @@
         prefix=""
         parent="world"
-        x="-0.5"
-        y="0.5"
-        z="0.5"
+        x="0"
+        y="1.0"
+        z="0.0"
         scale="0.0254"
     />
-    <xacro:include filename="$(find morpheus_teleop)/urdf/macros/double_sided_shelf.xacro" />
-    <xacro:double_sided_shelf
+    <xacro:include filename="$(find morpheus_teleop)/urdf/macros/double_level_shelf.xacro" />
+    <xacro:double_level_shelf
         prefix=""
         parent="world"
         x="0.0"
-        y="0.5"
-        z="0.5"
+        y="1.0"
+        z="0.0"
         scale="0.0254"
     />

File: morpheus_teleop/urdf/scenes/a_bot_keyhole_scene.xacro (robot description, xacro)
@@ -1,4 +1,4 @@
 <?xml version="1.0"?>
-<robot xmlns:xacro="http://www.ros.org/wiki/xacro" name="a_bot_double_sided_shelf_scene">
+<robot xmlns:xacro="http://www.ros.org/wiki/xacro" name="a_bot_keyhole_scene">
     <xacro:include filename="$(find morpheus_teleop)/urdf/scenes/a_bot_scene.xacro" />
     <xacro:include filename="$(find morpheus_teleop)/urdf/macros/table_2x8ft.xacro" />
@@ -11,6 +11,6 @@
         scale="0.0254"
     />
-    <xacro:include filename="$(find morpheus_teleop)/urdf/macros/double_sided_shelf.xacro" />
-    <xacro:double_sided_shelf
+    <xacro:include filename="$(find morpheus_teleop)/urdf/macros/keyhole.xacro" />
+    <xacro:keyhole
         prefix=""
         parent="world"

File: morpheus_teleop/urdf/scenes/a_bot_large_tunnel_scene.xacro (robot description, xacro)
@@ -1,4 +1,4 @@
 <?xml version="1.0"?>
-<robot xmlns:xacro="http://www.ros.org/wiki/xacro" name="a_bot_double_sided_shelf_scene">
+<robot xmlns:xacro="http://www.ros.org/wiki/xacro" name="a_bot_large_tunnel_scene">
     <xacro:include filename="$(find morpheus_teleop)/urdf/scenes/a_bot_scene.xacro" />
     <xacro:include filename="$(find morpheus_teleop)/urdf/macros/table_2x8ft.xacro" />
@@ -11,6 +11,6 @@
         scale="0.0254"
     />
-    <xacro:include filename="$(find morpheus_teleop)/urdf/macros/double_sided_shelf.xacro" />
-    <xacro:double_sided_shelf
+    <xacro:include filename="$(find morpheus_teleop)/urdf/macros/large_tunnel.xacro" />
+    <xacro:large_tunnel
         prefix=""
         parent="world"
