Commit message: Obstacles rewritten to be assemblies of sub-macros

File: morpheus_teleop/urdf/scenes/a_bot_trees_scene.xacro (robot description, xacro)
@@ -1,4 +1,4 @@
 <?xml version="1.0"?>
-<robot xmlns:xacro="http://www.ros.org/wiki/xacro" name="a_bot_double_sided_shelf_scene">
+<robot xmlns:xacro="http://www.ros.org/wiki/xacro" name="a_bot_trees_scene">
     <xacro:include filename="$(find morpheus_teleop)/urdf/scenes/a_bot_scene.xacro" />
     <xacro:include filename="$(find morpheus_teleop)/urdf/macros/table_2x8ft.xacro" />
@@ -7,14 +7,14 @@
         parent="world"
         x="-0.5"
-        y="0.5"
+        y="1.0"
         z="0.5"
         scale="0.0254"
     />
-    <xacro:include filename="$(find morpheus_teleop)/urdf/macros/double_sided_shelf.xacro" />
-    <xacro:double_sided_shelf
+    <xacro:include filename="$(find morpheus_teleop)/urdf/macros/trees.xacro" />
+    <xacro:trees
         prefix=""
         parent="world"
         x="0.0"
-        y="0.5"
+        y="0.6952"
         z="0.5"
         scale="0.0254"

Commit message: Twist->Pose converter done, cartesian control restored

File: morpheus_teleop/urdf/macros/Test_Block_1.xacro (robot description, xacro)
@@ -4,10 +4,4 @@
     params="x:=0 y:=0 z:=0 scale:=0.001 prefix parent">
     <link name="${prefix}test_block_1">
-        <contact>
-            <lateral_friction value="1.0"/>
-            <rolling_friction value="0.0"/>
-            <contact_cfm value="0.0"/>
-            <contact_erp value="1.0"/>
-        </contact>
         <inertial>
             <origin rpy="0 0 0" xyz="0.0 0.0 0.0"/>

File: morpheus_teleop/urdf/macros/bar_12in.xacro (robot description, xacro)
@@ -4,10 +4,4 @@
     params="x:=0 y:=0 z:=0 R:=0 P:=0 Y:=0 scale:=0.0254 prefix parent">
     <link name="${prefix}bar_12in">
-        <contact>
-            <lateral_friction value="1.0"/>
-            <rolling_friction value="0.05"/>
-            <contact_cfm value="0.0"/>
-            <contact_erp value="1.0"/>
-        </contact>
         <inertial>
             <origin rpy="0 0 0" xyz="${scale * 0.5} ${scale * 6.0} ${scale * 0.5}"/>

File: morpheus_teleop/urdf/macros/bar_4in.xacro (robot description, xacro)
@@ -4,10 +4,4 @@
     params="x:=0 y:=0 z:=0 R:=0 P:=0 Y:=0 scale:=0.0254 prefix parent">
     <link name="${prefix}bar_4in">
-        <contact>
-            <lateral_friction value="1.0"/>
-            <rolling_friction value="0.0"/>
-            <contact_cfm value="0.0"/>
-            <contact_erp value="1.0"/>
-        </contact>
         <inertial>
             <origin rpy="0 0 0" xyz="${scale * 0.5} ${scale * 0.5} ${scale * 2}"/>

File: morpheus_teleop/urdf/macros/block.xacro (robot description, xacro)
@@ -4,10 +4,4 @@
     params="x:=0 y:=0 z:=0 R:=0 P:=0 Y:=0 scale:=0.0254 prefix parent">
     <link name="${prefix}block">
-        <contact>
-            <lateral_friction value="1.0"/>
-            <rolling_friction value="0.0"/>
-            <contact_cfm value="0.0"/>
-            <contact_erp value="1.0"/>
-        </contact>
         <inertial>
             <origin rpy="0 0 0" xyz="0.0 0.0 0.0125"/>

File: morpheus_teleop/urdf/macros/dragon_simple.xacro (robot description, xacro)
@@ -4,10 +4,4 @@
     params="x:=0 y:=0 z:=0 R:=0 P:=0 Y:=0 scale:=0.0254 prefix parent">
     <link name="${prefix}dragon_simple">
-        <contact>
-            <lateral_friction value="1.0"/>
-            <rolling_friction value="0.0"/>
-            <contact_cfm value="0.0"/>
-            <contact_erp value="1.0"/>
-        </contact>
         <inertial>
             <origin rpy="0 0 0" xyz="${scale * 0.0} ${scale * 0.0} ${scale * 2}"/>

File: morpheus_teleop/urdf/macros/foam.xacro (robot description, xacro)
@@ -4,10 +4,4 @@
     params="x:=0 y:=0 z:=0 R:=0 P:=0 Y:=0 scale:=0.05 prefix parent">
     <link name="${prefix}foam">
-        <contact>
-            <lateral_friction value="1.0"/>
-            <rolling_friction value="0.0"/>
-            <contact_cfm value="0.0"/>
-            <contact_erp value="1.0"/>
-        </contact>
         <inertial>
             <origin rpy="0 0 0" xyz="0.0 0.0 0.0"/>

File: morpheus_teleop/urdf/macros/node2.xacro (robot description, xacro)
@@ -21,10 +21,4 @@
     </link>
     <link name="${prefix}PMA3">
-        <contact>
-            <lateral_friction value="1.0"/>
-            <rolling_friction value="0.05"/>
-            <contact_cfm value="0.0"/>
-            <contact_erp value="1.0"/>
-        </contact>
         <inertial>
             <origin rpy="0 0 0" xyz="0 0 0"/>

File: morpheus_teleop/urdf/macros/teapot.xacro (robot description, xacro)
@@ -4,10 +4,4 @@
     params="x:=0 y:=0 z:=0 scale:=0.05 prefix parent">
     <link name="${prefix}teapot">
-        <contact>
-            <lateral_friction value="1.0"/>
-            <rolling_friction value="0.0"/>
-            <contact_cfm value="0.0"/>
-            <contact_erp value="1.0"/>
-        </contact>
         <inertial>
             <origin rpy="0 0 0" xyz="0.0 0.0 0.0"/>

File: morpheus_teleop/urdf/macros/test_wall_1.xacro (robot description, xacro)
@@ -4,10 +4,4 @@
     params="x:=0 y:=0 z:=0 scale:=0.05 prefix parent">
     <link name="${prefix}test_wall_1">
-        <contact>
-            <lateral_friction value="1.0"/>
-            <rolling_friction value="0.0"/>
-            <contact_cfm value="0.0"/>
-            <contact_erp value="1.0"/>
-        </contact>
         <inertial>
             <origin rpy="0 0 0" xyz="0.0 0.0 0.0"/>

File: morpheus_teleop/urdf/macros/wall.xacro (robot description, xacro)
@@ -4,10 +4,4 @@
     params="x:=0 y:=0 z:=0 scale:=0.05 prefix parent">
     <link name="${prefix}wall">
-        <contact>
-            <lateral_friction value="1.0"/>
-            <rolling_friction value="0.0"/>
-            <contact_cfm value="0.0"/>
-            <contact_erp value="1.0"/>
-        </contact>
         <inertial>
             <origin rpy="0 0 0" xyz="0.0 0.0 0.0"/>

File: morpheus_teleop/urdf/macros/wall_4x12in.xacro (robot description, xacro)
@@ -4,10 +4,4 @@
     params="x:=0 y:=0 z:=0 R:=0 P:=0 Y:=0 scale:=0.0254 prefix parent">
     <link name="${prefix}wall_4x12in">
-        <contact>
-            <lateral_friction value="1.0"/>
-            <rolling_friction value="0.0"/>
-            <contact_cfm value="0.0"/>
-            <contact_erp value="1.0"/>
-        </contact>
         <inertial>
             <origin rpy="0 0 0" xyz="0.0 0.0 0.0"/>

File: morpheus_teleop/urdf/macros/wall_6x12in.xacro (robot description, xacro)
@@ -4,10 +4,4 @@
     params="x:=0 y:=0 z:=0 R:=0 P:=0 Y:=0 scale:=0.0254 prefix parent">
     <link name="${prefix}wall_6x12in">
-        <contact>
-            <lateral_friction value="1.0"/>
-            <rolling_friction value="0.0"/>
-            <contact_cfm value="0.0"/>
-            <contact_erp value="1.0"/>
-        </contact>
         <inertial>
             <origin rpy="0 0 0" xyz="${scale * 6} ${scale * 3} ${scale * 0.5}"/>

File: morpheus_teleop/urdf/scenes/trossen_scene.xacro (robot description, xacro)
@@ -15,4 +15,5 @@
         <origin xyz="0 0 0" rpy="0 0 0" />
     </xacro:trossen>
+    <link name="world" />
     <gazebo>
         <plugin name="ros_control" filename="libgazebo_ros_control.so">
