Commit message: Trossen main, UR5e main files added to launch robots in namespaces. Related collision issues debugged. URDF scenes modified to center robot at origin.

File: morpheus_description/urdf/macros/a_bot_macro.xacro (robot description, xacro)
@@ -1,6 +1,6 @@
 <?xml version="1.0"?>
 <robot xmlns:xacro="http://www.ros.org/wiki/xacro" name="a_bot">
-    <xacro:include filename="$(find homestri_description)/urdf/macros/ur5e_macro.xacro" />
-    <xacro:include filename="$(find homestri_description)/urdf/macros/d415_mount_macro.xacro" />
+    <xacro:include filename="$(find morpheus_description)/urdf/macros/ur5e_macro.xacro" />
+    <xacro:include filename="$(find morpheus_description)/urdf/macros/d415_mount_macro.xacro" />
     <xacro:include filename="$(find robotiq_2f_85_gripper_description)/urdf/robotiq_arg2f_85_macro.xacro" />
     <xacro:macro name="a_bot"

File: morpheus_description/urdf/macros/b_bot_macro.xacro (robot description, xacro)
@@ -1,6 +1,6 @@
 <?xml version="1.0"?>
 <robot xmlns:xacro="http://www.ros.org/wiki/xacro" name="b_bot">
-    <xacro:include filename="$(find homestri_description)/urdf/macros/ur5e_macro.xacro" />
-    <xacro:include filename="$(find homestri_description)/urdf/macros/d415_mount_macro.xacro" />
+    <xacro:include filename="$(find morpheus_description)/urdf/macros/ur5e_macro.xacro" />
+    <xacro:include filename="$(find morpheus_description)/urdf/macros/d415_mount_macro.xacro" />
     <xacro:include filename="$(find onrobot_rg2ft_description)/urdf/onrobot_rg2ft_macro.xacro" />
     <xacro:macro name="b_bot"

File: morpheus_description/urdf/macros/simple_pedestal_macro.xacro (robot description, xacro)
@@ -28,5 +28,5 @@
       <parent link="${parent}" />
       <child link="${prefix}pedestal" />
-      <origin xyz="0 0 ${height}" />
+      <origin xyz="0 0 0" />
     </joint>
   </xacro:macro>

File: morpheus_description/urdf/scenes/a_bot_scene.xacro (robot description, xacro)
@@ -4,15 +4,16 @@
         default="$(find ur_description)/config/ur5e/joint_limits.yaml" />
     <xacro:arg name="transmission_hw_interface" default="hardware_interface/PositionJointInterface" />
-    <xacro:include filename="$(find homestri_description)/urdf/macros/simple_pedestal_macro.xacro" />
-    <xacro:include filename="$(find homestri_description)/urdf/macros/a_bot_macro.xacro" />
+    <link name="world" />
+    <xacro:include filename="$(find morpheus_description)/urdf/macros/simple_pedestal_macro.xacro" />
+    <xacro:include filename="$(find morpheus_description)/urdf/macros/a_bot_macro.xacro" />
     <xacro:simple_pedestal
         prefix=""
         parent="world"
-        height="$(-0.0254 * 34.75)"
+        height="${0.0254 * 34.75}"
         radius="0.15"
     />
     <xacro:a_bot
         prefix=""
-        parent="pedestal"
+        parent="world"
         transmission_hw_interface="$(arg transmission_hw_interface)"
         joint_limits_parameters_file="$(arg joint_limits_parameters_file)"
@@ -20,5 +21,4 @@
         <origin xyz="0 0 0" rpy="0 0 0" />
     </xacro:a_bot>
-    <link name="world" />
     <gazebo>
         <plugin name="ros_control" filename="libgazebo_ros_control.so">

File: morpheus_description/urdf/scenes/b_bot_scene.xacro (robot description, xacro)
@@ -4,15 +4,16 @@
         default="$(find ur_description)/config/ur5e/joint_limits.yaml" />
     <xacro:arg name="transmission_hw_interface" default="hardware_interface/PositionJointInterface" />
-    <xacro:include filename="$(find homestri_description)/urdf/macros/simple_pedestal_macro.xacro" />
-    <xacro:include filename="$(find homestri_description)/urdf/macros/b_bot_macro.xacro" />
+    <link name="world" />
+    <xacro:include filename="$(find morpheus_description)/urdf/macros/simple_pedestal_macro.xacro" />
+    <xacro:include filename="$(find morpheus_description)/urdf/macros/b_bot_macro.xacro" />
     <xacro:simple_pedestal
         prefix=""
         parent="world"
-        height="$(-0.0254 * 34.75)"
+        height="${0.0254 * 34.75}"
         radius="0.15"
     />
     <xacro:b_bot
         prefix=""
-        parent="pedestal"
+        parent="world"
         transmission_hw_interface="$(arg transmission_hw_interface)"
         joint_limits_parameters_file="$(arg joint_limits_parameters_file)"
@@ -20,5 +21,4 @@
         <origin xyz="0 0 0" rpy="0 0 0" />
     </xacro:b_bot>
-    <link name="world" />
     <gazebo>
         <plugin name="ros_control" filename="libgazebo_ros_control.so">

File: morpheus_description/urdf/scenes/teapot_scene.xacro (robot description, xacro)
@@ -11,5 +11,5 @@
         scale="0.05"
     />
-    <xacro:include filename="$(find homestri_description)/urdf/macros/simple_pedestal_macro.xacro" />
+    <xacro:include filename="$(find morpheus_description)/urdf/macros/simple_pedestal_macro.xacro" />
     <xacro:simple_pedestal
         prefix=""

File: morpheus_description/urdf/scenes/trossen_scene.xacro (robot description, xacro)
@@ -9,10 +9,10 @@
     <xacro:arg name="external_urdf_loc" default=""/>
     <xacro:arg name="load_gazebo_configs" default="false"/>
-    <xacro:include filename="$(find homestri_description)/urdf/macros/simple_pedestal_macro.xacro" />
+    <xacro:include filename="$(find morpheus_description)/urdf/macros/simple_pedestal_macro.xacro" />
     <xacro:include filename="$(find morpheus_description)/urdf/macros/trossen_macro.xacro" />
     <xacro:simple_pedestal
         prefix=""
         parent="world"
-        height="$(-0.0254 * 34.75)"
+        height="$(0.0254 * 34.75)"
         radius="0.15"
     />

Commit message: Trossen description and teleop edited to move Trossen onto pedestal to avoid ground plane, keyboard control bugs fixed pending change of keyboard reader library

File: morpheus_description/urdf/macros/a_bot_macro.xacro (robot description, xacro)
@@ -18,5 +18,5 @@
             transmission_hw_interface="${transmission_hw_interface}"
         >
-            <origin xyz="0 0 0" rpy="0 0 0" />
+            <xacro:insert_block name="origin" />
         </xacro:ur5e>
         <xacro:d415_mount

File: morpheus_description/urdf/macros/b_bot_macro.xacro (robot description, xacro)
@@ -18,5 +18,5 @@
             transmission_hw_interface="${transmission_hw_interface}"
         >
-            <origin xyz="0 0 0" rpy="0 0 0" />
+            <xacro:insert_block name="origin" />
         </xacro:ur5e>
         <xacro:d415_mount

File: morpheus_description/urdf/macros/trossen_macro.xacro (robot description, xacro)
@@ -7,4 +7,12 @@
         parent
         *origin">
+        <xacro:arg name="robot_name" default="vx300s"/>
+        <xacro:arg name="base_link_frame" default="base_link"/>
+        <xacro:arg name="show_ar_tag" default="false"/>
+        <xacro:arg name="show_gripper_bar" default="true"/>
+        <xacro:arg name="show_gripper_fingers" default="true"/>
+        <xacro:arg name="use_world_frame" default="false"/>
+        <xacro:arg name="external_urdf_loc" default=""/>
+        <xacro:arg name="load_gazebo_configs" default="false"/>
         <xacro:vx300s
             prefix="${prefix}"
@@ -12,5 +20,13 @@
             tcp_offset="0.163"
         >
-            <origin xyz="0 0 0" rpy="0 0 0" />
+            <xacro:insert_block name="origin" />
+            <xacro:arg name="robot_name" value="${arg robot_name}"/>
+            <xacro:arg name="base_link_frame" value="${arg base_link_frame}"/>
+            <xacro:arg name="show_ar_tag" value="${arg show_ar_tag}"/>
+            <xacro:arg name="show_gripper_bar" value="${arg show_gripper_bar}"/>
+            <xacro:arg name="show_gripper_fingers" value="${arg show_gripper_fingers}"/>
+            <xacro:arg name="use_world_frame" value="${arg use_world_frame}"/>
+            <xacro:arg name="external_urdf_loc" value="${arg external_urdf_loc}"/>
+            <xacro:arg name="load_gazebo_configs" value="${arg load_gazebo_configs}"/>
         </xacro:vx300s>
     </xacro:macro>

File: morpheus_description/urdf/macros/vx300s_macro.xacro (robot description, xacro)
@@ -15,29 +15,29 @@
         <xacro:arg name="external_urdf_loc" default=""/>
         <xacro:arg name="load_gazebo_configs" default="false"/>
-        <xacro:macro name="vx300s_robot">
-            <xacro:include filename="$(find morpheus_description)/urdf/macros/vx300s.urdf.xacro">
-                <xacro:arg name="robot_name" value="${arg robot_name}"/>
-                <xacro:arg name="base_link_frame" value="${arg base_link_frame}"/>
-                <xacro:arg name="show_ar_tag" value="${arg show_ar_tag}"/>
-                <xacro:arg name="show_gripper_bar" value="${arg show_gripper_bar}"/>
-                <xacro:arg name="show_gripper_fingers" value="${arg show_gripper_fingers}"/>
-                <xacro:arg name="use_world_frame" value="${arg use_world_frame}"/>
-                <xacro:arg name="external_urdf_loc" value="${arg external_urdf_loc}"/>
-                <xacro:arg name="load_gazebo_configs" value="${arg load_gazebo_configs}"/>
-            </xacro:include>
-        </xacro:macro>
-        <xacro:vx300s_robot
-        >
-        </xacro:vx300s_robot>
-        <joint name="${prefix}trossen_base_joint" type="fixed">
-            <parent link="${parent}"/>
-            <child link="$(arg robot_name)/$(arg base_link_frame)"/>
-        </joint>
+        <xacro:include filename="$(find morpheus_description)/urdf/macros/vx300s.urdf.xacro">
+            <xacro:arg name="robot_name" value="${arg robot_name}"/>
+            <xacro:arg name="base_link_frame" value="${arg base_link_frame}"/>
+            <xacro:arg name="show_ar_tag" value="${arg show_ar_tag}"/>
+            <xacro:arg name="show_gripper_bar" value="${arg show_gripper_bar}"/>
+            <xacro:arg name="show_gripper_fingers" value="${arg show_gripper_fingers}"/>
+            <xacro:arg name="use_world_frame" value="${arg use_world_frame}"/>
+            <xacro:arg name="external_urdf_loc" value="${arg external_urdf_loc}"/>
+            <xacro:arg name="load_gazebo_configs" value="${arg load_gazebo_configs}"/>
+        </xacro:include>
+        <xacro:vx300s/>
+        <xacro:unless value="$(arg use_world_frame)">
+            <link name="world"/>
+            <joint name="${prefix}trossen_base_joint" type="fixed">
+                <parent link="${parent}"/>
+                <child link="$(arg robot_name)/$(arg base_link_frame)"/>
+                <xacro:insert_block name="origin" />
+            </joint>
+        </xacro:unless>
         <!-- Add an additional link to plan with. Oriented like the UR ee_link frame. -->
         <link name="${prefix}tcp_link" />
         <joint name="${prefix}tcp_joint" type="fixed">
-        <parent link="${prefix}vx300s/gripper_link" />
-        <child link="${prefix}tcp_link" />
-        <origin rpy="0 ${-pi/2} ${-pi/2}" xyz="0 0 ${tcp_offset}" />
+            <parent link="${prefix}vx300s/gripper_link" />
+            <child link="${prefix}tcp_link" />
+            <origin rpy="0 ${-pi/2} ${-pi/2}" xyz="0 0 ${tcp_offset}" />
         </joint>
     </xacro:macro>

File: morpheus_description/urdf/scenes/a_bot_node2_scene.xacro (robot description, xacro)
@@ -8,5 +8,5 @@
         x="${0.0254 * (-62)}"
         y="${0.0254 * 8.5}"
-        z="0"
+        z="${0.0254 * 34.75}"
         scale="1"
     />

File: morpheus_description/urdf/scenes/a_bot_scene.xacro (robot description, xacro)
@@ -19,5 +19,5 @@
         joint_limits_parameters_file="$(arg joint_limits_parameters_file)"
     >
-        <origin xyz="0 0 0" rpy="0 0 0" />
+        <origin xyz="0 0 ${0.0254 * 34.75}" rpy="0 0 0" />
     </xacro:a_bot>
     <gazebo>

File: morpheus_description/urdf/scenes/b_bot_node2_scene.xacro (robot description, xacro)
@@ -8,5 +8,5 @@
         x="${0.0254 * (-48)}"
         y="${0.0254 * 8.5}"
-        z="0"
+        z="${0.0254 * 34.75}"
         scale="1"
     />

File: morpheus_description/urdf/scenes/b_bot_scene.xacro (robot description, xacro)
@@ -19,5 +19,5 @@
         joint_limits_parameters_file="$(arg joint_limits_parameters_file)"
     >
-        <origin xyz="0 0 0" rpy="0 0 0" />
+        <origin xyz="0 0 ${0.0254 * 34.75}" rpy="0 0 0" />
     </xacro:b_bot>
     <gazebo>

File: morpheus_description/urdf/scenes/node2_scene.xacro (robot description, xacro)
@@ -7,5 +7,5 @@
         x="${0.0254 * (-48)}"
         y="${0.0254 * 8.5}"
-        z="0"
+        z="${0.0254 * 34.75}"
         scale="1"
     />

File: morpheus_description/urdf/scenes/trossen_node2_scene.xacro (robot description, xacro)
@@ -8,5 +8,5 @@
         x="${0.0254 * (-48)}"
         y="${0.0254 * 8.5}"
-        z="0"
+        z="${0.0254 * 34.75}"
         scale="1"
     />

File: morpheus_description/urdf/scenes/trossen_scene.xacro (robot description, xacro)
@@ -9,4 +9,5 @@
     <xacro:arg name="external_urdf_loc" default=""/>
     <xacro:arg name="load_gazebo_configs" default="false"/>
+    <link name="world" />
     <xacro:include filename="$(find morpheus_description)/urdf/macros/simple_pedestal_macro.xacro" />
     <xacro:include filename="$(find morpheus_description)/urdf/macros/trossen_macro.xacro" />
@@ -19,8 +20,7 @@
     <xacro:trossen
         prefix=""
-        parent="pedestal"
-        tcp_offfset="0"
+        parent="world"
     >
-        <origin xyz="0 0 0" rpy="0 0 0" />
+        <origin xyz="0 0 ${0.0254 * 34.75}" rpy="0 0 0" />
         <xacro:arg name="robot_name" value="${arg robot_name}"/>
         <xacro:arg name="base_link_frame" value="${arg base_link_frame}"/>
@@ -32,5 +32,4 @@
         <xacro:arg name="load_gazebo_configs" value="${arg load_gazebo_configs}"/>
     </xacro:trossen>
-    <link name="world" />
     <gazebo>
         <plugin name="ros_control" filename="libgazebo_ros_control.so">
