Commit message: HERA obstacle course addition in progress, Trossen scene geometry loading streamlined and made more flexible

File: morpheus_description/urdf/macros/simple_pedestal_macro.xacro (robot description, xacro)
@@ -28,5 +28,5 @@
       <parent link="${parent}" />
       <child link="${prefix}pedestal" />
-      <origin xyz="0 0 0" />
+      <origin xyz="0 0 ${height}" />
     </joint>
   </xacro:macro>

File: morpheus_description/urdf/macros/trossen_macro.xacro (robot description, xacro)
@@ -7,26 +7,11 @@
         parent
         *origin">
-        <xacro:arg name="robot_name" default="vx300s"/>
-        <xacro:arg name="base_link_frame" default="base_link"/>
-        <xacro:arg name="show_ar_tag" default="false"/>
-        <xacro:arg name="show_gripper_bar" default="true"/>
-        <xacro:arg name="show_gripper_fingers" default="true"/>
-        <xacro:arg name="use_world_frame" default="false"/>
-        <xacro:arg name="external_urdf_loc" default=""/>
-        <xacro:arg name="load_gazebo_configs" default="false"/>
+        <!-- tcp_offset is the summation of offsets from gripper_bar, ee_bar, and ee_gripper, i.e. the offset from ee_arm_link to ee_gripper_link -->
         <xacro:vx300s
             prefix="${prefix}"
             parent="${parent}"
-            tcp_offset="0.163"
+            tcp_offset="${0 + 0.025875 + 0.0385}"
         >
             <xacro:insert_block name="origin" />
-            <xacro:arg name="robot_name" value="${arg robot_name}"/>
-            <xacro:arg name="base_link_frame" value="${arg base_link_frame}"/>
-            <xacro:arg name="show_ar_tag" value="${arg show_ar_tag}"/>
-            <xacro:arg name="show_gripper_bar" value="${arg show_gripper_bar}"/>
-            <xacro:arg name="show_gripper_fingers" value="${arg show_gripper_fingers}"/>
-            <xacro:arg name="use_world_frame" value="${arg use_world_frame}"/>
-            <xacro:arg name="external_urdf_loc" value="${arg external_urdf_loc}"/>
-            <xacro:arg name="load_gazebo_configs" value="${arg load_gazebo_configs}"/>
         </xacro:vx300s>
     </xacro:macro>

File: morpheus_description/urdf/macros/ur5e_macro.xacro (robot description, xacro)
@@ -28,5 +28,5 @@
       <xacro:insert_block name="origin" />
     </joint>
-    <!-- Add an additional link to plan with. Oriented like the UR ee_link frame. -->
+    <!-- Add an additional link to plan with. Oriented like the Trossen ee_gripper_link frame. -->
     <link name="${prefix}tcp_link" />
     <joint name="${prefix}tcp_joint" type="fixed">

File: morpheus_description/urdf/macros/vx300s_macro.xacro (robot description, xacro)
@@ -5,25 +5,7 @@
         prefix
         parent
+        tcp_offset
         *origin">
-        <xacro:arg name="tcp_offset" default="0.04"/>
-        <xacro:arg name="robot_name" default="vx300s"/>
-        <xacro:arg name="base_link_frame" default="base_link"/>
-        <xacro:arg name="show_ar_tag" default="false"/>
-        <xacro:arg name="show_gripper_bar" default="true"/>
-        <xacro:arg name="show_gripper_fingers" default="true"/>
-        <xacro:arg name="use_world_frame" default="false"/>
-        <xacro:arg name="external_urdf_loc" default=""/>
-        <xacro:arg name="load_gazebo_configs" default="false"/>
-        <xacro:include filename="$(find morpheus_description)/urdf/macros/vx300s.urdf.xacro">
-            <xacro:arg name="robot_name" value="${arg robot_name}"/>
-            <xacro:arg name="base_link_frame" value="${arg base_link_frame}"/>
-            <xacro:arg name="show_ar_tag" value="${arg show_ar_tag}"/>
-            <xacro:arg name="show_gripper_bar" value="${arg show_gripper_bar}"/>
-            <xacro:arg name="show_gripper_fingers" value="${arg show_gripper_fingers}"/>
-            <xacro:arg name="use_world_frame" value="${arg use_world_frame}"/>
-            <xacro:arg name="external_urdf_loc" value="${arg external_urdf_loc}"/>
-            <xacro:arg name="load_gazebo_configs" value="${arg load_gazebo_configs}"/>
-        </xacro:include>
-        <xacro:vx300s/>
+        <xacro:include filename="$(find morpheus_description)/urdf/macros/vx300s.urdf.xacro"/>
         <xacro:unless value="$(arg use_world_frame)">
             <link name="world"/>
@@ -34,10 +16,10 @@
             </joint>
         </xacro:unless>
-        <!-- Add an additional link to plan with. Oriented like the UR ee_link frame. -->
+        <!-- Add an additional link to plan with. Identical to ee_gripper_link frame, included for consistency with HOMESTRI UR5e description. -->
         <link name="${prefix}tcp_link" />
         <joint name="${prefix}tcp_joint" type="fixed">
-            <parent link="${prefix}vx300s/gripper_link" />
+            <parent link="${prefix}vx300s/ee_arm_link" />
             <child link="${prefix}tcp_link" />
-            <origin rpy="0 ${-pi/2} ${-pi/2}" xyz="0 0 ${tcp_offset}" />
+            <origin rpy="0 0 0" xyz="${tcp_offset} 0 0" />
         </joint>
     </xacro:macro>

File: morpheus_description/urdf/scenes/trossen_scene.xacro (robot description, xacro)
@@ -1,21 +1,5 @@
 <?xml version="1.0"?>
 <robot xmlns:xacro="http://www.ros.org/wiki/xacro" name="trossen_scene">
-    <xacro:arg name="robot_name" default="vx300s"/>
-    <xacro:arg name="base_link_frame" default="base_link"/>
-    <xacro:arg name="show_ar_tag" default="false"/>
-    <xacro:arg name="show_gripper_bar" default="true"/>
-    <xacro:arg name="show_gripper_fingers" default="true"/>
-    <xacro:arg name="use_world_frame" default="false"/>
-    <xacro:arg name="external_urdf_loc" default=""/>
-    <xacro:arg name="load_gazebo_configs" default="false"/>
-    <link name="world" />
-    <xacro:include filename="$(find morpheus_description)/urdf/macros/simple_pedestal_macro.xacro" />
     <xacro:include filename="$(find morpheus_description)/urdf/macros/trossen_macro.xacro" />
-    <xacro:simple_pedestal
-        prefix=""
-        parent="world"
-        height="$(0.0254 * 34.75)"
-        radius="0.15"
-    />
     <xacro:trossen
         prefix=""
@@ -23,12 +7,4 @@
     >
         <origin xyz="0 0 ${0.0254 * 34.75}" rpy="0 0 0" />
-        <xacro:arg name="robot_name" value="${arg robot_name}"/>
-        <xacro:arg name="base_link_frame" value="${arg base_link_frame}"/>
-        <xacro:arg name="show_ar_tag" value="${arg show_ar_tag}"/>
-        <xacro:arg name="show_gripper_bar" value="${arg show_gripper_bar}"/>
-        <xacro:arg name="show_gripper_fingers" value="${arg show_gripper_fingers}"/>
-        <xacro:arg name="use_world_frame" value="${arg use_world_frame}"/>
-        <xacro:arg name="external_urdf_loc" value="${arg external_urdf_loc}"/>
-        <xacro:arg name="load_gazebo_configs" value="${arg load_gazebo_configs}"/>
     </xacro:trossen>
     <gazebo>
