Commit message: New HERA obstacle course xacro urdf based on box primitives instead of mesh, allowing concave collision detection

File: morpheus_description/urdf/macros/hera_obstacle_course.xacro (robot description, xacro)
@@ -1,39 +1,109 @@
 <?xml version="1.0"?>
 <robot name="hera_obstacle_course" xmlns:xacro="http://www.ros.org/wiki/xacro">
+    <xacro:include filename="$(find morpheus_description)/urdf/macros/box.xacro" />
     <xacro:macro name="hera_obstacle_course"
-        concave="yes"
         params="prefix parent *origin">
-        <link name="${prefix}hera_obstacle_course_link">
-            <inertial>
-                <origin xyz="-0.2 0.0 0.4"
-                    rpy="0 0 0" />
-                <mass value="0.0" />
-                <inertia ixx="4.3e-05" iyy="2.2e-05" izz="6.4e-05" ixy="3e-06" iyz="1e-06" ixz="0.0" />
-            </inertial>
-            <visual>
-                <origin xyz="0 0 0" rpy="0 0 ${pi}" />
-                <geometry>
-                    <mesh
-                        filename="package://morpheus_description/meshes/components/visual/HERAObstacleCourse.obj"
-                        scale="0.01 0.01 0.01" />
-                </geometry>
-                <material name="">
-                    <color rgba="0.3 0.3 0.3 1" />
-                  </material>
-            </visual>
-            <collision>
-                <origin xyz="0 0 0" rpy="0 0 ${pi}" />
-                <geometry>
-                    <mesh
-                        filename="package://morpheus_description/meshes/components/collision/HERAObstacleCourse.obj"
-                        scale="0.01 0.01 0.01" />
-                </geometry>
-            </collision>
-        </link>
-        <joint name="${prefix}hera_obstacle_course_joint" type="fixed">
+        <link name="${prefix}hera_obstacle_course_base_link"/>
+        <joint name="${prefix}hera_obstacle_course_base_link_joint" type="fixed">
             <parent link="${parent}" />
-            <child link="${prefix}hera_obstacle_course_link" />
+            <child link="${prefix}hera_obstacle_course_base_link" />
             <xacro:insert_block name="origin" />
         </joint>
+        <xacro:box
+            prefix="${prefix}hera_obstacle_course_floor_front_link"
+            parent="${prefix}hera_obstacle_course_base_link"
+            size="${0.015 * 1} ${0.44910} ${0.015 * 1}">
+            <origin xyz="${0.59055 - 0.015 * 0.5} ${0} ${0.015 * 0.5}" rpy="0 0 0" />
+        </xacro:box>
+        <xacro:box
+            prefix="${prefix}hera_obstacle_course_floor_left_link"
+            parent="${prefix}hera_obstacle_course_base_link"
+            size="${0.91440} ${0.015 * 1} ${0.015 * 1}">
+            <origin xyz="${-0.32385 + 0.91440 * 0.5} ${0.22455 - 0.015 * 0.5} ${0.015 * 0.5}" rpy="0 0 0" />
+        </xacro:box>
+        <xacro:box
+            prefix="${prefix}hera_obstacle_course_floor_right_link"
+            parent="${prefix}hera_obstacle_course_base_link"
+            size="${0.91440} ${0.015 * 1} ${0.015 * 1}">
+            <origin xyz="${-0.32385 + 0.91440 * 0.5} ${-0.22455 + 0.015 * 0.5} ${0.015 * 0.5}" rpy="0 0 0" />
+        </xacro:box>
+        <xacro:box
+            prefix="${prefix}hera_obstacle_course_floor_middle_link"
+            parent="${prefix}hera_obstacle_course_base_link"
+            size="${0.015 * 1} ${0.44910} ${0.015 * 1}">
+            <origin xyz="${0.15875 + 0.015 * 0.5} ${0} ${0.015 * 0.5}" rpy="0 0 0" />
+        </xacro:box>
+        <xacro:box
+            prefix="${prefix}hera_obstacle_course_floor_back_link"
+            parent="${prefix}hera_obstacle_course_base_link"
+            size="${0.015 * 1} ${0.44910} ${0.015 * 1}">
+            <origin xyz="${-0.32385 + 0.015 * 0.5} ${0} ${0.015 * 0.5}" rpy="0 0 0" />
+        </xacro:box>
+        <xacro:box
+            prefix="${prefix}hera_obstacle_course_wall_front_left_link"
+            parent="${prefix}hera_obstacle_course_base_link"
+            size="${0.015 * 1} ${0.015 * 1} ${0.60150}">
+            <origin xyz="${0.59055 - 0.015 * 0.5} ${0.22455 - 0.015 * 0.5} ${0.60150 * 0.5}" rpy="0 0 0" />
+        </xacro:box>
+        <xacro:box
+            prefix="${prefix}hera_obstacle_course_wall_front_right_link"
+            parent="${prefix}hera_obstacle_course_base_link"
+            size="${0.015 * 1} ${0.015 * 1} ${0.60150}">
+            <origin xyz="${0.59055 - 0.015 * 0.5} ${-0.22455 + 0.015 * 0.5} ${0.60150 * 0.5}" rpy="0 0 0" />
+        </xacro:box>
+        <xacro:box
+            prefix="${prefix}hera_obstacle_course_wall_middle_left_link"
+            parent="${prefix}hera_obstacle_course_base_link"
+            size="${0.015 * 1} ${0.015 * 1} ${0.60150}">
+            <origin xyz="${0.15875 + 0.015 * 0.5} ${0.22455 - 0.015 * 0.5} ${0.60150 * 0.5}" rpy="0 0 0" />
+        </xacro:box>
+        <xacro:box
+            prefix="${prefix}hera_obstacle_course_wall_middle_right_link"
+            parent="${prefix}hera_obstacle_course_base_link"
+            size="${0.015 * 1} ${0.015 * 1} ${0.60150}">
+            <origin xyz="${0.15875 + 0.015 * 0.5} ${-0.22455 + 0.015 * 0.5} ${0.60150 * 0.5}" rpy="0 0 0" />
+        </xacro:box>
+        <xacro:box
+            prefix="${prefix}hera_obstacle_course_wall_back_right_link"
+            parent="${prefix}hera_obstacle_course_base_link"
+            size="${0.015 * 1} ${0.015 * 1} ${0.60150}">
+            <origin xyz="${-0.32385 + 0.015 * 0.5} ${-0.22455 + 0.015 * 0.5} ${0.60150 * 0.5}" rpy="0 0 0" />
+        </xacro:box>
+        <xacro:box
+            prefix="${prefix}hera_obstacle_course_wall_back_post_link"
+            parent="${prefix}hera_obstacle_course_base_link"
+            size="${0.015 * 1} ${0.015 * 1} ${0.23320}">
+            <origin xyz="${-0.32385 + 0.31980 - 0.015 * 0.5} ${-0.22455 + 0.015 * 0.5} ${0.23320 * 0.5}" rpy="0 0 0" />
+        </xacro:box>
+        <xacro:box
+            prefix="${prefix}hera_obstacle_course_wall_back_crown_link"
+            parent="${prefix}hera_obstacle_course_base_link"
+            size="${0.31980} ${0.015 * 1} ${0.015 * 1}">
+            <origin xyz="${-0.32385 + 0.31980 * 0.5} ${-0.22455 + 0.015 * 0.5} ${0.23320 - 0.015 * 0.5}" rpy="0 0 0" />
+        </xacro:box>
+        <xacro:box
+            prefix="${prefix}hera_obstacle_course_roof_front_link"
+            parent="${prefix}hera_obstacle_course_base_link"
+            size="${0.015 * 1} ${0.44910} ${0.015 * 1}">
+            <origin xyz="${0.59055 - 0.015 * 0.5} ${0} ${0.60150 - 0.015 * 0.5}" rpy="0 0 0" />
+        </xacro:box>
+        <xacro:box
+            prefix="${prefix}hera_obstacle_course_roof_left_link"
+            parent="${prefix}hera_obstacle_course_base_link"
+            size="${0.43180} ${0.015 * 1} ${0.015 * 1}">
+            <origin xyz="${0.59055 - 0.43180 * 0.5} ${0.22455 - 0.015 * 0.5} ${0.60150 - 0.015 * 0.5}" rpy="0 0 0" />
+        </xacro:box>
+        <xacro:box
+            prefix="${prefix}hera_obstacle_course_roof_right_link"
+            parent="${prefix}hera_obstacle_course_base_link"
+            size="${0.91440} ${0.015 * 1} ${0.015 * 1}">
+            <origin xyz="${-0.32385 + 0.91440 * 0.5} ${-0.22455 + 0.015 * 0.5} ${0.60150 - 0.015 * 0.5}" rpy="0 0 0" />
+        </xacro:box>
+        <xacro:box
+            prefix="${prefix}hera_obstacle_course_roof_middle_link"
+            parent="${prefix}hera_obstacle_course_base_link"
+            size="${0.015 * 1} ${0.44910} ${0.015 * 1}">
+            <origin xyz="${0.15875 + 0.015 * 0.5} ${0} ${0.60150 - 0.015 * 0.5}" rpy="0 0 0" />
+        </xacro:box>
     </xacro:macro>
 </robot>

Commit message: Set Trossen scene names to vx300s in order to suppress warnings

File: morpheus_description/urdf/macros/hera_obstacle_course.xacro (robot description, xacro)
@@ -100,10 +100,4 @@
             <origin xyz="${-0.32385 + 0.91440 * 0.5} ${-0.22455 + 0.015 * 0.5} ${0.60150 - 0.015 * 0.5}" rpy="0 0 0" />
         </xacro:box>
-        <xacro:box
-            prefix="${prefix}hera_obstacle_course_roof_middle_link"
-            parent="${prefix}hera_obstacle_course_base_link"
-            size="${0.015 * 1} ${0.44910} ${0.015 * 1}">
-            <origin xyz="${0.15875 + 0.015 * 0.5} ${0} ${0.60150 - 0.015 * 0.5}" rpy="0 0 0" />
-        </xacro:box>
     </xacro:macro>
 </robot>

File: morpheus_description/urdf/scenes/trossen_hera_scene.xacro (robot description, xacro)
@@ -1,4 +1,4 @@
 <?xml version="1.0"?>
-<robot xmlns:xacro="http://www.ros.org/wiki/xacro" name="trossen_hera_scene">
+<robot xmlns:xacro="http://www.ros.org/wiki/xacro" name="vx300s">
     <xacro:include filename="$(find morpheus_description)/urdf/scenes/trossen_scene.xacro" />
     <xacro:include filename="$(find morpheus_description)/urdf/macros/hera_obstacle_course.xacro" />

File: morpheus_description/urdf/scenes/trossen_node2_external.xacro (robot description, xacro)
@@ -1,4 +1,4 @@
 <?xml version="1.0"?>
-<robot xmlns:xacro="http://www.ros.org/wiki/xacro" name="trossen_node2_scene">
+<robot xmlns:xacro="http://www.ros.org/wiki/xacro" name="vx300s">
     <xacro:arg name="robot_name" default="vx300s"/>
     <xacro:arg name="base_link_frame" default="base_link"/>

File: morpheus_description/urdf/scenes/trossen_node2_scene.xacro (robot description, xacro)
@@ -1,4 +1,4 @@
 <?xml version="1.0"?>
-<robot xmlns:xacro="http://www.ros.org/wiki/xacro" name="trossen_node2_scene">
+<robot xmlns:xacro="http://www.ros.org/wiki/xacro" name="vx300s">
     <xacro:include filename="$(find morpheus_description)/urdf/scenes/trossen_scene.xacro" />
     <xacro:include filename="$(find morpheus_description)/urdf/macros/node2_table.xacro" />

File: morpheus_description/urdf/scenes/trossen_scene.xacro (robot description, xacro)
@@ -1,4 +1,4 @@
 <?xml version="1.0"?>
-<robot xmlns:xacro="http://www.ros.org/wiki/xacro" name="trossen_scene">
+<robot xmlns:xacro="http://www.ros.org/wiki/xacro" name="vx300s">
     <xacro:include filename="$(find morpheus_description)/urdf/macros/trossen_macro.xacro" />
     <xacro:trossen

Commit message: Updated URDF, SRDF, and all references to SRDF in Trossen launch files to add table and visual indicators of the pick and place goals for HERA

File: morpheus_description/urdf/macros/hera_obstacle_course.xacro (robot description, xacro)
@@ -2,4 +2,6 @@
 <robot name="hera_obstacle_course" xmlns:xacro="http://www.ros.org/wiki/xacro">
     <xacro:include filename="$(find morpheus_description)/urdf/macros/box.xacro" />
+    <xacro:include filename="$(find morpheus_description)/urdf/macros/hera_pick_goal.xacro" />
+    <xacro:include filename="$(find morpheus_description)/urdf/macros/hera_place_goal.xacro" />
     <xacro:macro name="hera_obstacle_course"
         params="prefix parent *origin">
@@ -100,4 +102,25 @@
             <origin xyz="${-0.32385 + 0.91440 * 0.5} ${-0.22455 + 0.015 * 0.5} ${0.60150 - 0.015 * 0.5}" rpy="0 0 0" />
         </xacro:box>
+        <xacro:hera_pick_goal
+            prefix="${prefix}hera_obstacle_course_easy_pick_goal"
+            parent="${prefix}hera_obstacle_course_base_link"
+            radius="${0.0254 * 1.0}"
+            length="${0.0254 * 0.5}">
+            <origin xyz="${0.59055 - 0.015 * 1.5} ${0} ${0.60150 - 0.015 * 0.5}" rpy="0 ${pi/2} 0" />
+        </xacro:hera_pick_goal>
+        <xacro:hera_pick_goal
+            prefix="${prefix}hera_obstacle_course_hard_pick_goal"
+            parent="${prefix}hera_obstacle_course_base_link"
+            radius="${0.0254 * 1.0}"
+            length="${0.0254 * 0.5}">
+            <origin xyz="${-0.32385 + 0.31980 * 0.5} ${-0.22455 + 0.015 * 0.5 + (0.0254 * -4)} ${0.015 * 1.5}" rpy="0 0 0" />
+        </xacro:hera_pick_goal>
+        <xacro:hera_place_goal
+            prefix="${prefix}hera_obstacle_course_place_goal"
+            parent="${prefix}hera_obstacle_course_base_link"
+            radius="${0.0254 * 1.0}"
+            length="${0.0254 * 0.5}">
+            <origin xyz="${0.0254 * 10} 0.0 ${0.015 * 0.5}" rpy="0 0 0" />
+        </xacro:hera_place_goal>
     </xacro:macro>
 </robot>

File: morpheus_description/urdf/scenes/trossen_hera_scene.xacro (robot description, xacro)
@@ -1,5 +1,7 @@
 <?xml version="1.0"?>
 <robot xmlns:xacro="http://www.ros.org/wiki/xacro" name="vx300s">
+    <!-- Trossen scene (already calls the Trossen macro) -->
     <xacro:include filename="$(find morpheus_description)/urdf/scenes/trossen_scene.xacro" />
+    <!-- Hera version of the obstacle course -->
     <xacro:include filename="$(find morpheus_description)/urdf/macros/hera_obstacle_course.xacro" />
     <xacro:hera_obstacle_course
@@ -7,6 +9,20 @@
         parent="world"
     >
-        <origin xyz="0 0 ${0.0254 * 34.75}" rpy="0 0 0" />
+        <origin xyz="${0.0254 * (-0.5)} 0 ${0.0254 * 34.75}" rpy="0 0 0" />
     </xacro:hera_obstacle_course>
     <!-- scale=0.0254 meters/inch -->
+    <!-- Note the obstacle course is moved 0.5 inches to the right from its original position -->
+    <!-- This was done so that the Trossen robot remains fully within the obstacle course at rest -->
+    <!-- Otherwise, the elbow would extend slightly outside the allowed bounds at rest -->
+    <!-- Table -->
+    <xacro:include filename="$(find morpheus_description)/urdf/macros/hera_table.xacro" />
+    <xacro:hera_table
+        prefix=""
+        parent="world"
+        x="${(0.59055 + (-0.32385)) / 2 + 0.0254 * (-0.5)}"
+        y="${0.22455 + (0.0254 * -12)}"
+        z="${0.0254 * 34.75}"
+    />
+    <!-- The table is centered such that the obstacle course fits neatly within its dimensions (3'x2') -->
+    <!-- Adjustments to the obstacle course position therefore must also be applied to the table -->
 </robot>
