Commit message: Restore collision for hera goal objects

File: morpheus_description/urdf/macros/hera_pick_goal.xacro (robot description, xacro)
@@ -14,7 +14,7 @@
       </visual>
       <collision>
-        <origin xyz="0 0 -1000000" rpy="0 0 0"/>
+        <origin xyz="0 0 0" rpy="0 0 0"/>
         <geometry>
-          <cylinder radius="0" length="0"/>
+          <cylinder radius="${radius}" length="${length}"/>
         </geometry>
       </collision>

File: morpheus_description/urdf/macros/hera_place_goal.xacro (robot description, xacro)
@@ -14,7 +14,7 @@
       </visual>
       <collision>
-        <origin xyz="0 0 -1000000" rpy="0 0 0"/>
+        <origin xyz="0 0 0" rpy="0 0 0"/>
         <geometry>
-          <cylinder radius="0" length="0"/>
+          <cylinder radius="${radius}" length="${length}"/>
         </geometry>
       </collision>
